File: hw/sch_pcb/SPACEDOS02A_PCB01A/SPACEDOS02A_PCB01A.kicad_pcb (KiCad board)
At the start: 2 copper layers, 48.2 x 93.5 mm, 92 parts, among them J1 HEADER_2x01, J19 HEADER_2x01_PARALLEL, J2 HEADER_2x01_PARALLEL, J22 HEADER_2x03, J3 HEADER_2x01_PARALLEL, J4 HEADER_1x01, J5 HEADER_1x01, J6 HEADER_1x01, J7 HEADER_1x01, M1 HOLE, M10 BMI-S-204-F, M2 HOLE, M3 HOLE, M4 HOLE, M6 BMI-S-210-F, M8 BMI-S-204-F, M9 BMI-S-204-F, U1 OPA2314, U10 ATMEGA1284P-AU, U11 PCF85263A, U2 OPA2314, U3 ISL21080DIH312Z-TK 1V25, U4 TS7211, U5 TS5A4594, U8 TPS613222ADBV, Y2 ABS07-120-32.768KHZ-T

Commit message: Edit
Parts:
- removed J1: HEADER_2x01, Mlab_Pin_Headers:Straight_1x02
- added BT1: BX0037, Mlab_Batery:BX0037, F.Cu at (19.1, -52.2)
- added C22: 10uF, Mlab_R:SMD-0805, B.Cu at (58.6, -63.0)
- added C25: 100nF, Mlab_R:SMD-0805, B.Cu at (51.1, -68.4)
- added C30: 100nF, Mlab_R:SMD-0805, B.Cu at (58.6, -61.2)
- added J8: SD_Card, Mlab_CON:MCC-SD, B.Cu at (18.4, -96.0)
- added R14: 100, Mlab_R:SMD-0805, B.Cu at (55.1, -63.0)
- added R16: 100, Mlab_R:SMD-0805, B.Cu at (51.1, -66.6)
- added R17: 100, Mlab_R:SMD-0805, B.Cu at (58.6, -59.4)
- added R18: 100, Mlab_R:SMD-0805, B.Cu at (47.6, -68.4)
- added U6: AT24CS64-SSHM, Package_SO:SOIC-8_3.9x4.9mm_P1.27mm, B.Cu at (56.7, -66.6)
- C1, C10, C11, C12, C13, C14, C15, C16, C17, C18, C19, C2, C20, C21, C23, C24, C26, C27, C28, C29, C3, C31, C32, C34, C35, C36, C39, C4, C40, C42, C43, C44, C47, C5, C50, C52, C54, C55, C6, C7, C8, C9, D3, F2, J22, L1, L3, M6, M9, R1, R10, R11, R12, R13, R15, R19, R2, R20, R21, R22, R23, R3, R4, R5, R6, R7, R8, R9, U1, U10, U11, U2, U3, U4, U5, U8, Y2: moved to B.Cu
- D1: footprint Mlab_D:HAMAMATSU_S11773-02 -> Mlab_D:HAMAMATSU_S2744-09
- J19, J2, J3, J4, J5, J6, J7: moved to F.Cu
- moved M8 224.8 mm to (200.1, -202.7)
- moved M2 198.0 mm to (236.1, -27.9)
- moved M4 195.6 mm to (239.4, -6.60)
- moved M1 176.7 mm to (247.4, -27.3)
- moved M10 165.9 mm to (208.3, -127.6)
- moved M3 153.7 mm to (238.3, -17.4)
- moved J5 74.3 mm to (5.46, -52.7)
- moved J7 74.3 mm to (5.46, -55.2)
- moved F2 73.8 mm to (5.71, -68.8)
- moved C55 72.8 mm to (6.22, -76.6), turned to 180 degrees
- moved C29 71.8 mm to (6.73, -73.3)
- moved J19 71.8 mm to (6.73, -57.8), turned to 0 degrees
- moved J2 71.8 mm to (6.73, -60.3)
- moved J3 71.8 mm to (6.73, -65.4)
- moved R15 69.3 mm to (7.99, -27.0)
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Connections:
- U10 pad 41: (no net) -> /cpu/SD_VDD
- U10 pad 42: (no net) -> /cpu/SD_VDD
- U10 pad 43: (no net) -> /cpu/SD_VDD
- U10 pad 44: (no net) -> /cpu/PB4
Routing:
- net PA1: track 105.2 -> 92.5 mm, vias 2 -> 1
- net +3V3: track 199.5 -> 193.1 mm
- net PA0: track 29.3 -> 23.2 mm
- net Net-(C18-Pad1): track 30.1 -> 25.8 mm
- net Net-(C18-Pad2): track 7.06 -> 4.42 mm
- net GND: vias 162 -> 160
- net /A: vias 0 -> 1
- removed copper zone on B.Cu, net GND
- removed copper zone on F.Cu, net GND
Other:
- board size 48.2 x 93.5 mm -> 38 x 110 mm
