File: hw/sch_pcb/SPACEDOS02A_PCB01A/SPACEDOS02A_PCB01A.kicad_pcb (KiCad board)
At the start: 2 copper layers, 38 x 110 mm, 101 parts, among them J19 HEADER_2x01_PARALLEL, J2 HEADER_2x01_PARALLEL, J22 HEADER_2x03, J3 HEADER_2x01_PARALLEL, J4 HEADER_1x01, J5 HEADER_1x01, J6 HEADER_1x01, J7 HEADER_1x01, J8 SD_Card, M1 HOLE, M10 BMI-S-204-F, M2 HOLE, M3 HOLE, M4 HOLE, M6 BMI-S-210-F, M8 BMI-S-204-F, M9 BMI-S-204-F, U1 OPA2314, U10 ATMEGA1284P-AU, U11 PCF85263A, U2 OPA2314, U3 ISL21080DIH312Z-TK 1V25, U4 TS7211, U5 TS5A4594, U6 AT24CS64-SSHM, U8 TPS613222ADBV, Y2 ABS07-120-32.768KHZ-T

Commit message: Edit
Parts:
- removed J8: SD_Card, Mlab_CON:MCC-SD
- removed M10, M9: BMI-S-204-F, RF_Shielding:Laird_Technologies_BMI-S-204-F_32.00x32.00mm
- added J1: SD_Card-Connector, Mlab_CON:MCC-SD, F.Cu at (14.2, -145.0)
- added REF**: SD_TE_2041021, Mlab_CON:FPS009-4200-0, F.Cu at (61.5, -75.9)
- BT1: footprint Mlab_Batery:BX0037 -> Mlab_Batery:BX0037_nez_sroubu
- M8: value BMI-S-204-F -> BMI-S-210-F; footprint RF_Shielding:Laird_Technologies_BMI-S-204-F_32.00x32.00mm -> RF_Shielding:Laird_Technologies_BMI-S-210-F_44.00x30.50mm
- moved M8 224.9 mm to (19.3, -68.8)
- moved R17 111.5 mm to (11.2, -160.3), turned to 270 degrees
- moved C22 106.6 mm to (15.5, -160.5), turned to 90 degrees
- moved R14 102.9 mm to (21.1, -160.1), turned to 270 degrees
- moved R18 100.5 mm to (6.10, -160.0), turned to 270 degrees
- moved C25 99.2 mm to (13.5, -160.2), turned to 90 degrees
- moved R16 98.9 mm to (18.5, -160.1), turned to 270 degrees
- moved J5 50.4 mm to (17.5, -101.6)
- moved U6 49.7 mm to (8.38, -54.9), turned to 90 degrees
- moved J4 47.3 mm to (17.5, -99.1)
- moved J6 46.9 mm to (15.0, -101.6)
- moved C30 46.7 mm to (12.4, -54.3), turned to 270 degrees
- moved J7 44.8 mm to (15.0, -99.1)
- moved J19 42.5 mm to (7.37, -100.3), turned to 90 degrees
- moved J2 40.4 mm to (12.4, -100.3), turned to 0 degrees
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Routing:
- net GND: track 106.2 -> 83.4 mm, vias 160 -> 174
- net /cpu/PD2: track 16.0 -> 0.00 mm, vias 2 -> 0
- net /cpu/RST#: track 14.1 -> 0.00 mm, vias 2 -> 0
- net PA1: track 92.5 -> 106.5 mm, vias 1 -> 2
- net /cpu/PC1: track 23.7 -> 37.4 mm
- net /cpu/TX0: track 12.3 -> 0.00 mm
- net /cpu/PC0: track 25.8 -> 38.0 mm
- net /cpu/PD3: track 11.1 -> 0.00 mm, vias 2 -> 0
- net /cpu/RX0: track 9.89 -> 0.00 mm
- net +3V3: track 193.1 -> 202.5 mm
- net /power/3: track 5.06 -> 0.00 mm
- net /A: track 17.2 -> 19.1 mm, vias 1 -> 0
- net Net-(J1-Pad2): vias 0 -> 1
Other:
- board text removed: "SPACEDOS01B_PCB01A"

Commit message: Edit PCB
Parts:
- removed REF**: SD_TE_2041021, Mlab_CON:FPS009-4200-0
- added J10: HEADER_1x01, Mlab_Pin_Headers:Straight_1x01, F.Cu at (66.0, -102.5)
- added J11: HEADER_1x01, Mlab_Pin_Headers:Straight_1x01, F.Cu at (66.0, -98.9)
- added J12: HEADER_1x01, Mlab_Pin_Headers:Straight_1x01, F.Cu at (69.7, -102.5)
- added J13: HEADER_1x01, Mlab_Pin_Headers:Straight_1x01, F.Cu at (69.7, -98.9)
- added J8: HEADER_1x01, Mlab_Pin_Headers:Straight_1x01, F.Cu at (62.3, -102.5)
- added J9: HEADER_1x01, Mlab_Pin_Headers:Straight_1x01, F.Cu at (62.3, -98.9)
- moved C34 1.14 mm to (16.8, -54.8), turned to 90 degrees
- moved R23 0.37 mm to (17.8, -51.2)
Connections:
- J1 pad 4: /cpu/SD_VDD -> (no net)
- R14 pad 1: /cpu/PB4 -> (no net)
- R16 pad 1: /cpu/PB5 -> (no net)
- R17 pad 1: /cpu/PB7 -> (no net)
- R18 pad 1: /cpu/PB6 -> (no net)
Routing:
- net /cpu/RST#: track 0.00 -> 54.6 mm, vias 0 -> 2
- net /cpu/RX0: track 0.00 -> 50.7 mm, vias 0 -> 2
- net +3V3: track 202.5 -> 204.0 mm

Commit message: Edit PCB
Parts:
- J10, J11, J12, J13, J8, J9: moved to B.Cu
- moved J12 47.2 mm to (22.6, -106.4)
- moved J11 46.5 mm to (20.1, -106.4)
- moved J9 37.9 mm to (25.1, -106.4)
- moved J13 37.7 mm to (32.8, -106.4)
- moved J10 36.0 mm to (30.2, -106.4)
- moved J8 34.8 mm to (27.7, -106.4)
- moved F2 27.4 mm to (30.5, -80.6)
- moved C36 27.2 mm to (32.5, -80.6)
- moved Y2 25.1 mm to (7.87, -80.0), turned to 0 degrees
- moved C55 24.6 mm to (29.8, -83.6)
- moved R21 23.5 mm to (8.95, -60.2)
- moved D3 23.3 mm to (29.2, -87.1)
- moved C29 21.9 mm to (26.7, -82.3)
- moved U11 19.3 mm to (8.38, -74.9), turned to 270 degrees
- moved C47 16.8 mm to (11.4, -76.8), turned to 90 degrees
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Routing:
- net /cpu/SD_VDD: track 0.00 -> 55.8 mm, vias 0 -> 1
- net /cpu/PB5: track 5.50 -> 59.5 mm, vias 0 -> 1
- net /cpu/PB6: track 8.97 -> 60.2 mm
- net /cpu/PB7: track 8.25 -> 58.6 mm, vias 0 -> 1
- net /cpu/PB4: track 0.00 -> 49.7 mm, vias 0 -> 1
- net /cpu/TX0: track 0.00 -> 43.5 mm, vias 0 -> 2
- net /cpu/PC1: track 37.4 -> 20.2 mm, vias 2 -> 0
- net /cpu/PC0: track 38.0 -> 22.1 mm
- net GND: track 83.4 -> 72.5 mm, vias 174 -> 171
- net +3V3: track 204.0 -> 194.4 mm
- net Net-(C29-Pad1): track 8.04 -> 0.00 mm
- net PA0: track 23.2 -> 29.3 mm
- net PA1: track 106.5 -> 112.1 mm
- net /cpu/RX0: track 50.7 -> 46.1 mm
- net /cpu/RST#: track 54.6 -> 51.2 mm
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
Commit message: Edit PCB
Routing:
- net GND: track 72.5 -> 99.8 mm
Changed lines of the file:
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@@
     (thickness 1.6)
     (drawings 25)
-    (tracks 665)
+    (tracks 667)
     (zones 0)
     (modules 105)
@@
   )
   (setup
-    (last_trace_width 0.4)
+    (last_trace_width 0.25)
     (user_trace_width 0.3)
     (user_trace_width 0.4)
@@
   (segment (start 10.4941 -64.5961) (end 9.906 -64.008) (width 0.4) (layer B.Cu) (net 1) (status 20))
   (segment (start 12.7963 -64.5961) (end 10.4941 -64.5961) (width 0.4) (layer B.Cu) (net 1) (status 10))
+  (segment (start 1.574 -133.709) (end 27.874 -133.709) (width 0.25) (layer F.Cu) (net 1))
+  (segment (start 0.574 -133.709) (end 1.574 -133.709) (width 0.25) (layer F.Cu) (net 1))
   (segment (start 22.2183 -9.4056) (end 22.2183 -7.8181) (width 0.4) (layer B.Cu) (net 2) (status 30))
   (segment (start 20.3133 -7.6581) (end 22.0583 -7.6581) (width 0.4) (layer B.Cu) (net 2) (status 30))

Commit message: Edit PCB
Parts:
- removed M1, M2, M3, M4: HOLE, Mlab_Mechanical:MountingHole_3mm
- moved F2 13.4 mm to (19.1, -87.6), turned to 90 degrees
- moved D3 11.6 mm to (18.3, -83.3), turned to 180 degrees
- moved C36 8.41 mm to (24.2, -81.8), turned to 0 degrees
- moved C29 4.80 mm to (23.1, -85.5)
- moved C32 4.77 mm to (28.5, -65.0)
- moved C35 4.45 mm to (28.5, -67.3)
- moved L3 4.24 mm to (28.7, -62.7)
- moved C55 4.10 mm to (26.4, -85.9), turned to 270 degrees
- moved J4 2.54 mm to (12.4, -101.6)
- moved J5 2.54 mm to (12.4, -99.1)
- moved U8 2.14 mm to (30.7, -59.4)
- moved C50 2.01 mm to (30.5, -53.8)
- moved C42 1.94 mm to (30.5, -56.1)
- moved C52 1.14 mm to (31.5, -50.3)
- moved C54 0.38 mm to (28.6, -49.8)
Connections:
- J4 pad 1: /cpu/PD3 -> /cpu/PC4
- J5 pad 1: /cpu/PD2 -> /cpu/PC3
- U10 pad 11: /cpu/PD2 -> (no net)
- U10 pad 12: /cpu/PD3 -> (no net)
- U10 pad 22: (no net) -> /cpu/PC3
- U10 pad 23: (no net) -> /cpu/PC4
Routing:
- net /cpu/PC4: track 0.00 -> 38.1 mm, vias 0 -> 1
- net /cpu/PC3: track 0.00 -> 35.2 mm, vias 0 -> 1
- net /power/3: track 0.00 -> 16.5 mm
- net Net-(C29-Pad1): track 0.00 -> 10.6 mm
- net PA0: track 29.3 -> 34.9 mm
- net Net-(C18-Pad1): track 25.8 -> 30.1 mm
- net /cpu/PC1: track 20.2 -> 24.0 mm
- net +3V3: track 194.4 -> 198.0 mm
- net Net-(C18-Pad2): track 4.42 -> 7.06 mm
- net /cpu/PB5: track 59.5 -> 61.7 mm
- net PA1: track 112.1 -> 114.1 mm
- net /cpu/TX0: track 43.5 -> 45.4 mm
- net Net-(C42-Pad1): track 8.01 -> 6.72 mm
- net +5V: track 46.1 -> 45.0 mm
- net Net-(J1-Pad2): vias 1 -> 0
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- added copper zone on B.Cu, net GND
- added copper zone on F.Cu, net GND
Other:
- board text added: "PC4,3"

Commit message: Edit
Parts:
- added C33: 10uF, Mlab_R:SMD-0805, B.Cu at (21.3, -192.0)
- added C37: 100nF, Mlab_R:SMD-0805, B.Cu at (21.3, -189.5)
- added J14: HEADER_1x01, Mlab_Pin_Headers:Straight_1x01, F.Cu at (27.7, -146.6)
- added J15: HEADER_1x01, Mlab_Pin_Headers:Straight_1x01, F.Cu at (25.1, -146.6)
- added J16: HEADER_1x01, Mlab_Pin_Headers:Straight_1x01, F.Cu at (30.2, -146.6)
- added J17: HEADER_1x01, Mlab_Pin_Headers:Straight_1x01, F.Cu at (20.1, -146.6)
- added J18: HEADER_1x01, Mlab_Pin_Headers:Straight_1x01, F.Cu at (22.6, -146.6)
- added J20: HEADER_1x01, Mlab_Pin_Headers:Straight_1x01, F.Cu at (32.8, -146.6)
- added J21: HEADER_1x01, Mlab_Pin_Headers:Straight_1x01, F.Cu at (27.7, -196.6)
- added J23: HEADER_1x01, Mlab_Pin_Headers:Straight_1x01, F.Cu at (25.1, -196.6)
- added J24: HEADER_1x01, Mlab_Pin_Headers:Straight_1x01, F.Cu at (30.2, -196.6)
- added J25: HEADER_1x01, Mlab_Pin_Headers:Straight_1x01, F.Cu at (20.1, -196.6)
- added J26: HEADER_1x01, Mlab_Pin_Headers:Straight_1x01, F.Cu at (22.6, -196.6)
- added J27: HEADER_1x01, Mlab_Pin_Headers:Straight_1x01, F.Cu at (32.8, -196.6)
- added J28: SD_Card-FPS009-4200-0, Mlab_CON:FPS009-4200-0, B.Cu at (20.3, -150.4)
- added R24: 100, Mlab_R:SMD-0805, B.Cu at (14.7, -189.9)
- added R25: 100, Mlab_R:SMD-0805, B.Cu at (17.3, -189.9)
- added R26: 100, Mlab_R:SMD-0805, B.Cu at (24.9, -189.9)
- added R27: 100, Mlab_R:SMD-0805, B.Cu at (30.0, -189.9)
- J1: moved to B.Cu
- moved R18 29.4 mm to (26.7, -139.0)
- moved R17 23.9 mm to (21.6, -138.9)
- moved R14 23.1 mm to (11.7, -138.9)
- moved J1 21.8 mm to (18.5, -123.7), turned to 180 degrees
- moved C25 21.7 mm to (17.7, -138.9), turned to 180 degrees
- moved R16 21.6 mm to (14.2, -138.9)
- moved C22 18.4 mm to (17.7, -142.2), turned to 180 degrees
Connections:
- C22 pad 1: /cpu/SD_VDD -> /cpu/SD_VDD2
- C25 pad 1: /cpu/SD_VDD -> /cpu/SD_VDD2
- J1 pad 4: (no net) -> /cpu/SD_VDD2
- R14 pad 1: (no net) -> Net-(J14-Pad1)
- R16 pad 1: (no net) -> Net-(J15-Pad1)
- R17 pad 1: (no net) -> Net-(J17-Pad1)
- R18 pad 1: (no net) -> Net-(J18-Pad1)
Routing:
- net Net-(J14-Pad1): track 0.00 -> 22.2 mm
- net /cpu/SD_VDD2: track 0.00 -> 20.9 mm, vias 0 -> 1
- net Net-(J21-Pad1): track 0.00 -> 19.5 mm
- net Net-(J15-Pad1): track 0.00 -> 16.9 mm
- net /cpu/SD_VDD3: track 0.00 -> 16.2 mm, vias 0 -> 1
- net Net-(J23-Pad1): track 0.00 -> 14.4 mm
- net Net-(J26-Pad1): track 0.00 -> 10.4 mm
- net Net-(J18-Pad1): track 0.00 -> 8.93 mm
- net Net-(J25-Pad1): track 0.00 -> 7.71 mm
- net Net-(J17-Pad1): track 0.00 -> 7.36 mm
- net /cpu/RST#: track 51.3 -> 53.9 mm
- net Net-(J28-Pad1): track 0.00 -> 2.49 mm
- net Net-(J28-Pad2): track 0.00 -> 2.47 mm
- net Net-(J28-Pad7): track 0.00 -> 2.45 mm
- net Net-(J28-Pad5): track 0.00 -> 2.42 mm
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Other:
- board size 38 x 110 mm -> 38 x 200 mm
- board text added: "SPACEDOS02A_PCB01A"
- board text removed: "PD2"
- board text removed: "PD3"
- board text removed: "RX0"
- board text removed: "TX0"
