File: hw/sch_pcb/SPACEDOS02A_PCB01A/SPACEDOS02A_PCB01A.sch (KiCad schematic (older format))
At the start: 53 parts, among them M1 HOLE, M10 BMI-S-204-F, M2 HOLE, M3 HOLE, M4 HOLE, M6 BMI-S-210-F, M8 BMI-S-204-F, M9 BMI-S-204-F, U1 OPA2314, U2 OPA2314, U3 ISL21080DIH312Z-TK 1V25, U4 TS7211, U5 TS5A4594

Commit message: Edit
Parts:
- D1: footprint Mlab_D:HAMAMATSU_S11773-02 -> Mlab_D:HAMAMATSU_S2744-09
Changed lines of the file:
@@
 F 0 "D1" H 1350 4450 50  0000 C CNN
 F 1 "S11773-02" H 1650 4550 50  0000 C CNN
-F 2 "Mlab_D:HAMAMATSU_S11773-02" H 1650 4350 50  0001 C CNN
+F 2 "Mlab_D:HAMAMATSU_S2744-09" H 1650 4350 50  0001 C CNN
 F 3 "~" H 1650 4350 50  0001 C CNN
 	1    1700 4350

Commit message: Edit
Parts:
- removed M10, M9: BMI-S-204-F, RF_Shielding:Laird_Technologies_BMI-S-204-F_32.00x32.00mm, symbol MLAB_MECHANICAL:HOLE
- M8: value BMI-S-204-F -> BMI-S-210-F; footprint RF_Shielding:Laird_Technologies_BMI-S-204-F_32.00x32.00mm -> RF_Shielding:Laird_Technologies_BMI-S-210-F_44.00x30.50mm
Changed lines of the file:
@@
 EESchema Schematic File Version 4
 LIBS:SPACEDOS02A_PCB01A-cache
-EELAYER 26 0
+EELAYER 29 0
 EELAYER END
 $Descr A4 11693 8268
@@
 P 9200 750
 F 0 "M8" V 9100 750 60  0000 C CNN
-F 1 "BMI-S-204-F" H 9200 650 60  0001 C CNN
-F 2 "RF_Shielding:Laird_Technologies_BMI-S-204-F_32.00x32.00mm" H 9200 750 60  0001 C CNN
+F 1 "BMI-S-210-F" H 9200 650 60  0001 C CNN
+F 2 "RF_Shielding:Laird_Technologies_BMI-S-210-F_44.00x30.50mm" H 9200 750 60  0001 C CNN
 F 3 "" H 9200 750 60  0000 C CNN
 	1    9200 750
@@
 	9200 650  9200 700
 $Comp
-L MLAB_MECHANICAL:HOLE M9
-U 1 1 5C81F263
-P 8800 750
-F 0 "M9" V 8700 750 60  0000 C CNN
-F 1 "BMI-S-204-F" H 8800 650 60  0001 C CNN
-F 2 "RF_Shielding:Laird_Technologies_BMI-S-204-F_32.00x32.00mm" H 8800 750 60  0001 C CNN
-F 3 "" H 8800 750 60  0000 C CNN
-	1    8800 750
-	0    -1   -1   0
-$EndComp
-$Comp
-L MLAB_MECHANICAL:HOLE M10
-U 1 1 5C81F2E9
-P 9000 750
-F 0 "M10" V 8900 750 60  0000 C CNN
-F 1 "BMI-S-204-F" H 9000 650 60  0001 C CNN
-F 2 "RF_Shielding:Laird_Technologies_BMI-S-204-F_32.00x32.00mm" H 9000 750 60  0001 C CNN
-F 3 "" H 9000 750 60  0000 C CNN
-	1    9000 750
-	0    -1   -1   0
-$EndComp
-Wire Wire Line
-	9200 650  9000 650
-Wire Wire Line
-	8800 650  8800 700
-Connection ~ 9200 650
-Wire Wire Line
-	9000 700  9000 650
-Connection ~ 9000 650
-Wire Wire Line
-	9000 650  8800 650
-$Comp
 L Device:D_Photo D1

Commit message: Edit PCB
Parts:
- removed M1, M2, M3, M4: HOLE, Mlab_Mechanical:MountingHole_3mm, symbol MLAB_MECHANICAL:HOLE
Other:
- moved on the sheet: M6, M8
Changed lines of the file:
@@
 $EndDescr
-$Comp
-L MLAB_MECHANICAL:HOLE M1
-U 1 1 5C4AF3DA
-P 10200 750
-F 0 "M1" V 10100 750 60  0000 C CNN
-F 1 "HOLE" H 10200 650 60  0001 C CNN
-F 2 "Mlab_Mechanical:MountingHole_3mm" H 10200 750 60  0001 C CNN
-F 3 "" H 10200 750 60  0000 C CNN
-	1    10200 750
-	0    -1   -1   0
-$EndComp
-$Comp
-L MLAB_MECHANICAL:HOLE M2
-U 1 1 549D7628
-P 10400 750
-F 0 "M2" V 10300 750 60  0000 C CNN
-F 1 "HOLE" H 10400 650 60  0001 C CNN
-F 2 "Mlab_Mechanical:MountingHole_3mm" H 10400 750 60  0001 C CNN
-F 3 "" H 10400 750 60  0000 C CNN
-	1    10400 750
-	0    -1   -1   0
-$EndComp
-$Comp
-L MLAB_MECHANICAL:HOLE M3
-U 1 1 5B3D3F17
-P 10600 750
-F 0 "M3" V 10500 750 60  0000 C CNN
-F 1 "HOLE" H 10600 650 60  0001 C CNN
-F 2 "Mlab_Mechanical:MountingHole_3mm" H 10600 750 60  0001 C CNN
-F 3 "" H 10600 750 60  0000 C CNN
-	1    10600 750
-	0    -1   -1   0
-$EndComp
-$Comp
-L MLAB_MECHANICAL:HOLE M4
-U 1 1 5B3D3F18
-P 10800 750
-F 0 "M4" V 10700 750 60  0000 C CNN
-F 1 "HOLE" H 10800 650 60  0001 C CNN
-F 2 "Mlab_Mechanical:MountingHole_3mm" H 10800 750 60  0001 C CNN
-F 3 "" H 10800 750 60  0000 C CNN
-	1    10800 750
-	0    -1   -1   0
-$EndComp
 $Comp
 L power:GND #PWR03
@@
 	11000 650  10800 650
 Wire Wire Line
-	10200 650  10200 700
-Wire Wire Line
-	10400 700  10400 650
-Connection ~ 10400 650
-Wire Wire Line
 	10600 700  10600 650
-Connection ~ 10600 650
 Wire Wire Line
 	10800 700  10800 650
@@
 Text Notes 10100 1000 0    60   ~ 0
 MOUNTING HOLES
-Wire Wire Line
-	10400 650  10200 650
-Wire Wire Line
-	10600 650  10400 650
 Wire Wire Line
 	10800 650  10600 650
@@
 L MLAB_MECHANICAL:HOLE M6
 U 1 1 5B47DBA2
-P 10000 750
-F 0 "M6" V 9900 750 60  0000 C CNN
-F 1 "BMI-S-210-F" H 10000 650 60  0001 C CNN
-F 2 "Mlab_Mechanical:BMI-S-210-F" H 10000 750 60  0001 C CNN
-F 3 "" H 10000 750 60  0000 C CNN
-	1    10000 750
+P 10600 750
+F 0 "M6" V 10500 750 60  0000 C CNN
+F 1 "BMI-S-210-F" H 10600 650 60  0001 C CNN
+F 2 "Mlab_Mechanical:BMI-S-210-F" H 10600 750 60  0001 C CNN
+F 3 "" H 10600 750 60  0000 C CNN
+	1    10600 750
 	0    -1   -1   0
 $EndComp
-Connection ~ 10200 650
-Wire Wire Line
-	10000 700  10000 650
-Wire Wire Line
-	10000 650  10200 650
 Wire Notes Line
 	9700 600  9700 1000
 Wire Notes Line
-	9700 600  11100 600
-Wire Notes Line
 	9700 1000 11100 1000
-Connection ~ 10000 650
 Wire Wire Line
 	6750 4450 7450 4450
@@
 L MLAB_MECHANICAL:HOLE M8
 U 1 1 5C71374D
-P 9200 750
-F 0 "M8" V 9100 750 60  0000 C CNN
-F 1 "BMI-S-210-F" H 9200 650 60  0001 C CNN
-F 2 "RF_Shielding:Laird_Technologies_BMI-S-210-F_44.00x30.50mm" H 9200 750 60  0001 C CNN
-F 3 "" H 9200 750 60  0000 C CNN
-	1    9200 750
+P 10800 750
+F 0 "M8" V 10700 750 60  0000 C CNN
+F 1 "BMI-S-210-F" H 10800 650 60  0001 C CNN
+F 2 "RF_Shielding:Laird_Technologies_BMI-S-210-F_44.00x30.50mm" H 10800 750 60  0001 C CNN
+F 3 "" H 10800 750 60  0000 C CNN
+	1    10800 750
 	0    -1   -1   0
 $EndComp
-Wire Wire Line
-	9200 650  9200 700
 $Comp
 L Device:D_Photo D1
@@
 Wire Wire Line
 	1000 4350 1500 4350
-Wire Wire Line
-	9200 650  10000 650
+Wire Notes Line
+	9700 600  11100 600
 $EndSCHEMATC

Commit message: Edit
Parts:
- C1: UST_ID (none) -> 5c70984412875079b91f8869
- C10, C11, C12, C13, C14, C16, C2, C20: UST_ID (none) -> 5c70984712875079b91f8b4c
- C15: UST_ID (none) -> 5c70984712875079b91f8b47
- C17, C3: UST_ID (none) -> 5c70984712875079b91f8b52
- C18: UST_ID (none) -> 5c70984712875079b91f8b46
- C19: UST_ID (none) -> 5c70984812875079b91f8ba6
- C21, C23, C4, C6, C7, C8, C9: UST_ID (none) -> 5c70984812875079b91f8bbd
- C24: UST_ID (none) -> 5c70984712875079b91f8b50
- C5: UST_ID (none) -> 5c70984712875079b91f8b9f
- D1: value S11773-02 -> S2744-09
- M6, M8: UST_ID (none) -> 5c70984312875079b91f873d
- R1: UST_ID (none) -> 5c70984512875079b91f896d
- R10, R8: UST_ID (none) -> 5c70984512875079b91f898c
- R11, R15, R19, R22, R9: UST_ID (none) -> 5c70984612875079b91f8995
- R12, R7: UST_ID (none) -> 5c70984612875079b91f899f
- R13: UST_ID (none) -> 5c70984612875079b91f8990
- R2, R3, R4, R5: UST_ID (none) -> 5c70984512875079b91f8986
- R6: UST_ID (none) -> 5c70984712875079b91f8aae
- U1, U2: UST_ID (none) -> 5c70984412875079b91f879b
- U3: UST_ID (none) -> 5c70984712875079b91f8b7a
- U4: UST_ID (none) -> 5c70984712875079b91f8b5b
- U5: UST_ID (none) -> 5c70984612875079b91f8a0d
Changed lines of the file:
@@
 F 2 "Mlab_IO:SOIC-8_3.9x4.9mm_Pitch1.27mm" H 2400 4850 60  0001 C CNN
 F 3 "" H 2941 4729 60  0000 L CNN
+F 4 "5c70984412875079b91f879b" H 2400 4850 50  0001 C CNN "UST_ID"
 	1    2400 4850
 	1    0    0    1
@@
 F 2 "Mlab_IO:SOIC-8_3.9x4.9mm_Pitch1.27mm" H 6150 5050 60  0001 C CNN
 F 3 "" H 6691 4929 60  0000 L CNN
+F 4 "5c70984412875079b91f879b" H 6150 5050 50  0001 C CNN "UST_ID"
 	1    6150 5050
 	1    0    0    1
@@
 F 2 "Mlab_R:SMD-0805" H 1788 5050 50  0001 C CNN
 F 3 "~" H 1750 5200 50  0001 C CNN
+F 4 "5c70984712875079b91f8b52" H 1750 5200 50  0001 C CNN "UST_ID"
 	1    1750 5200
 	1    0    0    -1
@@
 F 2 "Mlab_R:SMD-0805" H 2438 4000 50  0001 C CNN
 F 3 "~" H 2400 4150 50  0001 C CNN
+F 4 "5c70984712875079b91f8b9f" H 2400 4150 50  0001 C CNN "UST_ID"
 	1    2400 4150
 	0    1    1    0
@@
 F 2 "Mlab_R:SMD-0805" V 2330 3750 50  0001 C CNN
 F 3 "~" H 2400 3750 50  0001 C CNN
+F 4 "5c70984712875079b91f8aae" H 2400 3750 50  0001 C CNN "UST_ID"
 	1    2400 3750
 	0    1    1    0
@@
 F 2 "Mlab_R:SMD-0805" V 3280 5050 50  0001 C CNN
 F 3 "~" H 3350 5050 50  0001 C CNN
+F 4 "5c70984612875079b91f899f" H 3350 5050 50  0001 C CNN "UST_ID"
 	1    3350 5050
 	-1   0    0    1
@@
 F 2 "Mlab_R:SMD-0805" H 3188 4700 50  0001 C CNN
 F 3 "~" H 3150 4850 50  0001 C CNN
+F 4 "5c70984712875079b91f8b4c" H 3150 4850 50  0001 C CNN "UST_ID"
 	1    3150 4850
 	0    1    1    0
@@
 F 2 "Mlab_R:SMD-0805" V 4080 5700 50  0001 C CNN
 F 3 "~" H 4150 5700 50  0001 C CNN
+F 4 "5c70984612875079b91f8995" H 4150 5700 50  0001 C CNN "UST_ID"
 	1    4150 5700
 	0    1    1    0
@@
 F 2 "Mlab_R:SMD-0805" H 4188 5900 50  0001 C CNN
 F 3 "~" H 4150 6050 50  0001 C CNN
+F 4 "5c70984712875079b91f8b47" H 4150 6050 50  0001 C CNN "UST_ID"
 	1    4150 6050
 	0    1    1    0
@@
 F 2 "Mlab_R:SMD-0805" V 3630 6250 50  0001 C CNN
 F 3 "~" H 3700 6250 50  0001 C CNN
+F 4 "5c70984512875079b91f898c" H 3700 6250 50  0001 C CNN "UST_ID"
 	1    3700 6250
 	1    0    0    -1
@@
 F 2 "Mlab_R:SMD-0805" H 5038 4800 50  0001 C CNN
 F 3 "~" H 5000 4950 50  0001 C CNN
+F 4 "5c70984712875079b91f8b4c" H 5000 4950 50  0001 C CNN "UST_ID"
 	1    5000 4950
 	0    1    1    0
@@
 F 2 "Mlab_R:SMD-0805" V 5330 4950 50  0001 C CNN
 F 3 "~" H 5400 4950 50  0001 C CNN
+F 4 "5c70984512875079b91f898c" H 5400 4950 50  0001 C CNN "UST_ID"
 	1    5400 4950
 	0    1    1    0
@@
 F 2 "Package_TO_SOT_SMD:SOT-23-5_HandSoldering" H 7200 5150 50  0001 C CNN
 F 3 "http://www.analog.com/media/en/technical-documentation/data-sheets/OP179_279.pdf" H 7200 5350 50  0001 C CNN
+F 4 "5c70984712875079b91f8b5b" H 7200 5150 50  0001 C CNN "UST_ID"
 	1    7200 5150
 	1    0    0    -1
@@
 F 2 "Package_TO_SOT_SMD:SOT-23-5_HandSoldering" H 8300 5100 60  0001 C CNN
 F 3 "" H 8300 5100 60  0001 C CNN
+F 4 "5c70984612875079b91f8a0d" H 7900 4400 50  0001 C CNN "UST_ID"
 	1    7900 4400
 	1    0    0    -1
@@
 F 2 "Mlab_R:SMD-0805" V 7630 5150 50  0001 C CNN
 F 3 "~" H 7700 5150 50  0001 C CNN
+F 4 "5c70984612875079b91f899f" H 7700 5150 50  0001 C CNN "UST_ID"
 	1    7700 5150
 	0    1    1    0
@@
 F 2 "Mlab_R:SMD-0805" V 7580 3700 50  0001 C CNN
 F 3 "~" H 7650 3700 50  0001 C CNN
+F 4 "5c70984612875079b91f8990" H 7650 3700 50  0001 C CNN "UST_ID"
 	1    7650 3700
 	0    1    1    0
@@
 F 2 "Mlab_R:SMD-0805" H 8288 3750 50  0001 C CNN
 F 3 "~" H 8250 3900 50  0001 C CNN
+F 4 "5c70984812875079b91f8ba6" H 8250 3900 50  0001 C CNN "UST_ID"
 	1    8250 3900
 	1    0    0    -1
@@
 F 2 "Mlab_R:SMD-0805" H 5638 5200 50  0001 C CNN
 F 3 "~" H 5600 5350 50  0001 C CNN
+F 4 "5c70984712875079b91f8b52" H 5600 5350 50  0001 C CNN "UST_ID"
 	1    5600 5350
 	1    0    0    -1
@@
 F 2 "Mlab_R:SMD-0805" H 6138 3900 50  0001 C CNN
 F 3 "~" H 6100 4050 50  0001 C CNN
+F 4 "5c70984712875079b91f8b46" H 6100 4050 50  0001 C CNN "UST_ID"
 	1    6100 4050
 	0    1    1    0
@@
 F 2 "Mlab_R:SMD-0805" V 6030 4400 50  0001 C CNN
 F 3 "~" H 6100 4400 50  0001 C CNN
+F 4 "5c70984612875079b91f8995" H 6100 4400 50  0001 C CNN "UST_ID"
 	1    6100 4400
 	0    1    1    0
@@
 F 2 "Mlab_R:SMD-0805" V 2330 950 50  0001 C CNN
 F 3 "~" H 2400 950 50  0001 C CNN
+F 4 "5c70984512875079b91f8986" H 2400 950 50  0001 C CNN "UST_ID"
 	1    2400 950
 	0    1    1    0
@@
 F 2 "Mlab_C:TantalC_SizeC_Reflow" H 1438 1000 50  0001 C CNN
 F 3 "~" H 1400 1150 50  0001 C CNN
+F 4 "5c70984412875079b91f8869" H 1400 1150 50  0001 C CNN "UST_ID"
 	1    1400 1150
 	1    0    0    -1
@@
 F 2 "Mlab_R:SMD-0805" H 1888 1000 50  0001 C CNN
 F 3 "~" H 1850 1150 50  0001 C CNN
+F 4 "5c70984812875079b91f8bbd" H 1850 1150 50  0001 C CNN "UST_ID"
 	1    1850 1150
 	1    0    0    -1
@@
 F 2 "Mlab_R:SMD-0805" H 2788 1000 50  0001 C CNN
 F 3 "~" H 2750 1150 50  0001 C CNN
+F 4 "5c70984812875079b91f8bbd" H 2750 1150 50  0001 C CNN "UST_ID"
 	1    2750 1150
 	1    0    0    -1
@@
 F 2 "Mlab_R:SMD-0805" H 3238 1000 50  0001 C CNN
 F 3 "~" H 3200 1150 50  0001 C CNN
+F 4 "5c70984712875079b91f8b4c" H 3200 1150 50  0001 C CNN "UST_ID"
 	1    3200 1150
 	1    0    0    -1
@@
 F 2 "Mlab_R:SMD-0805" V 2330 1600 50  0001 C CNN
 F 3 "~" H 2400 1600 50  0001 C CNN
+F 4 "5c70984512875079b91f8986" H 2400 1600 50  0001 C CNN "UST_ID"
 	1    2400 1600
 	0    1    1    0
@@
 F 2 "Mlab_R:SMD-0805" H 2788 1650 50  0001 C CNN
 F 3 "~" H 2750 1800 50  0001 C CNN
+F 4 "5c70984812875079b91f8bbd" H 2750 1800 50  0001 C CNN "UST_ID"
 	1    2750 1800
 	1    0    0    -1
@@
 F 2 "Mlab_R:SMD-0805" H 3238 1650 50  0001 C CNN
 F 3 "~" H 3200 1800 50  0001 C CNN
+F 4 "5c70984712875079b91f8b4c" H 3200 1800 50  0001 C CNN "UST_ID"
 	1    3200 1800
 	1    0    0    -1
@@
 F 2 "Mlab_R:SMD-0805" V 2330 2250 50  0001 C CNN
 F 3 "~" H 2400 2250 50  0001 C CNN
+F 4 "5c70984512875079b91f8986" H 2400 2250 50  0001 C CNN "UST_ID"
 	1    2400 2250
 	0    1    1    0
@@
 F 2 "Mlab_R:SMD-0805" H 2788 2300 50  0001 C CNN
 F 3 "~" H 2750 2450 50  0001 C CNN
+F 4 "5c70984812875079b91f8bbd" H 2750 2450 50  0001 C CNN "UST_ID"
 	1    2750 2450
 	1    0    0    -1
@@
 F 2 "Mlab_R:SMD-0805" H 3238 2300 50  0001 C CNN
 F 3 "~" H 3200 2450 50  0001 C CNN
+F 4 "5c70984712875079b91f8b4c" H 3200 2450 50  0001 C CNN "UST_ID"
 	1    3200 2450
 	1    0    0    -1
@@
 F 2 "Mlab_R:SMD-0805" V 2330 2900 50  0001 C CNN
 F 3 "~" H 2400 2900 50  0001 C CNN
+F 4 "5c70984512875079b91f8986" H 2400 2900 50  0001 C CNN "UST_ID"
 	1    2400 2900
 	0    1    1    0
@@
 F 2 "Mlab_R:SMD-0805" H 2788 2950 50  0001 C CNN
 F 3 "~" H 2750 3100 50  0001 C CNN
+F 4 "5c70984812875079b91f8bbd" H 2750 3100 50  0001 C CNN "UST_ID"
 	1    2750 3100
 	1    0    0    -1
@@
 F 2 "Mlab_R:SMD-0805" H 3238 2950 50  0001 C CNN
 F 3 "~" H 3200 3100 50  0001 C CNN
+F 4 "5c70984712875079b91f8b4c" H 3200 3100 50  0001 C CNN "UST_ID"
 	1    3200 3100
 	1    0    0    -1
@@
 F 2 "Package_TO_SOT_SMD:SOT-23" H 5100 1300 50  0001 C CIN
 F 3 "http://www.intersil.com/content/dam/Intersil/documents/fn75/fn7599.pdf" H 4600 1550 50  0001 C CIN
+F 4 "5c70984712875079b91f8b7a" H 4600 1550 50  0001 C CNN "UST_ID"
 	1    4600 1550
 	1    0    0    -1
@@
 F 2 "Mlab_R:SMD-0805" H 5038 1600 50  0001 C CNN
 F 3 "" H 5000 1750 50  0001 C CNN
+F 4 "5c70984712875079b91f8b4c" H 5000 1750 50  0001 C CNN "UST_ID"
 	1    5000 1750
 	1    0    0    -1
@@
 F 2 "Mlab_Mechanical:BMI-S-210-F" H 10600 750 60  0001 C CNN
 F 3 "" H 10600 750 60  0000 C CNN
+F 4 "5c70984312875079b91f873d" H 10600 750 50  0001 C CNN "UST_ID"
 	1    10600 750
 	0    -1   -1   0
@@
 F 2 "Mlab_R:SMD-0805" V 9780 3800 50  0001 C CNN
 F 3 "~" H 9850 3800 50  0001 C CNN
+F 4 "5c70984512875079b91f896d" H 9850 3800 50  0001 C CNN "UST_ID"
 	1    9850 3800
 	0    1    1    0
@@
 F 2 "Mlab_R:SMD-0805" V 1080 6750 50  0001 C CNN
 F 3 "~" H 1150 6750 50  0001 C CNN
+F 4 "5c70984612875079b91f8995" H 1150 6750 50  0001 C CNN "UST_ID"
 	1    1150 6750
 	0    1    1    0
@@
 F 2 "Mlab_R:SMD-0805" H 1388 6850 50  0001 C CNN
 F 3 "~" H 1350 7000 50  0001 C CNN
+F 4 "5c70984812875079b91f8bbd" H 1350 7000 50  0001 C CNN "UST_ID"
 	1    1350 7000
 	1    0    0    -1
@@
 F 2 "Mlab_R:SMD-0805" V 1480 6750 50  0001 C CNN
 F 3 "~" H 1550 6750 50  0001 C CNN
+F 4 "5c70984612875079b91f8995" H 1550 6750 50  0001 C CNN "UST_ID"
 	1    1550 6750
 	0    1    1    0
@@
 F 2 "Mlab_R:SMD-0805" H 1788 6850 50  0001 C CNN
 F 3 "~" H 1750 7000 50  0001 C CNN
+F 4 "5c70984812875079b91f8bbd" H 1750 7000 50  0001 C CNN "UST_ID"
 	1    1750 7000
 	1    0    0    -1
@@
 F 2 "Mlab_R:SMD-0805" V 2530 6750 50  0001 C CNN
 F 3 "~" H 2600 6750 50  0001 C CNN
+F 4 "5c70984612875079b91f8995" H 2600 6750 50  0001 C CNN "UST_ID"
 	1    2600 6750
 	0    1    1    0
@@
 F 2 "Mlab_R:SMD-0805" H 2888 6850 50  0001 C CNN
 F 3 "~" H 2850 7000 50  0001 C CNN
+F 4 "5c70984712875079b91f8b50" H 2850 7000 50  0001 C CNN "UST_ID"
 	1    2850 7000
 	1    0    0    -1
@@
 F 2 "Mlab_R:SMD-0805" H 2238 6850 50  0001 C CNN
 F 3 "" H 2200 7000 50  0001 C CNN
+F 4 "5c70984712875079b91f8b4c" H 2200 7000 50  0001 C CNN "UST_ID"
 	1    2200 7000
 	1    0    0    -1
@@
 F 2 "RF_Shielding:Laird_Technologies_BMI-S-210-F_44.00x30.50mm" H 10800 750 60  0001 C CNN
 F 3 "" H 10800 750 60  0000 C CNN
+F 4 "5c70984312875079b91f873d" H 10800 750 50  0001 C CNN "UST_ID"
 	1    10800 750
 	0    -1   -1   0
@@
 P 1700 4350
 F 0 "D1" H 1350 4450 50  0000 C CNN
-F 1 "S11773-02" H 1650 4550 50  0000 C CNN
+F 1 "S2744-09" H 1650 4550 50  0000 C CNN
 F 2 "Mlab_D:HAMAMATSU_S2744-09" H 1650 4350 50  0001 C CNN
 F 3 "~" H 1650 4350 50  0001 C CNN
