File: hw/sch_pcb/SPACEDOS02A_PCB01A/cpu.sch (KiCad schematic (older format))
At the start: 33 parts, among them J19 HEADER_2x01_PARALLEL, J22 HEADER_2x03, J4 HEADER_1x01, J5 HEADER_1x01, J6 HEADER_1x01, J7 HEADER_1x01, J8 SD_Card, U10 ATMEGA1284P-AU, U11 PCF85263A, U6 AT24CS64-SSHM, Y2 ABS07-120-32.768KHZ-T

Commit message: Edit
Parts:
- removed J8: SD_Card, Mlab_CON:MCC-SD, symbol Connector:SD_Card
- added J1: SD_Card-Connector, Mlab_CON:MCC-SD, symbol MLAB_CONNECTORS:SD_Card-Connector
Connections:
- net GND: now also J1.12 (SHELL1), J1.3 (VSS), J1.6 (VSS)
- net SD_VDD: now also J1.4 (VDD)
- net at R14.2: now also J1.1 (CD/DAT3)
- net at R16.2: now also J1.2 (CMD)
- net at R17.2: now also J1.5 (CLK)
- net at R18.2: now also J1.7 (DAT0)
Changed lines of the file:
@@
 EESchema Schematic File Version 4
 LIBS:SPACEDOS02A_PCB01A-cache
-EELAYER 26 0
+EELAYER 29 0
 EELAYER END
 $Descr A4 11693 8268
@@
 SD_VDD
 $Comp
-L Connector:SD_Card J8
-U 1 1 5CC65CD6
-P 2650 5500
-F 0 "J8" H 2650 6165 50  0000 C CNN
-F 1 "SD_Card" H 2650 6074 50  0000 C CNN
-F 2 "Mlab_CON:MCC-SD" H 2650 5500 50  0001 C CNN
-F 3 "http://portal.fciconnect.com/Comergent//fci/drawing/10067847.pdf" H 2650 5500 50  0001 C CNN
-	1    2650 5500
-	1    0    0    -1
-$EndComp
-$Comp
 L power:GND #PWR0126
 U 1 1 5CC665A4
@@
 Wire Wire Line
 	3550 5600 3700 5600
-Wire Wire Line
-	3700 5600 3700 5700
-Wire Wire Line
-	3550 5700 3700 5700
-Connection ~ 3700 5700
-Wire Wire Line
-	3700 5700 3700 6250
 $Comp
 L SPACEDOS02A_PCB01A-rescue:C-device-DATALOGGER01A-rescue-CCP2019V01A-rescue-SPACEDOS01A_PCB01A-rescue-SPACEDOS01B_PCB01A-rescue C22
@@
 Wire Wire Line
 	6850 2800 6950 2800
+$Comp
+L MLAB_CONNECTORS:SD_Card-Connector J1
+U 1 1 5CCD373E
+P 2650 5500
+F 0 "J1" H 2650 6165 50  0000 C CNN
+F 1 "SD_Card-Connector" H 2650 6074 50  0000 C CNN
+F 2 "Mlab_CON:MCC-SD" H 2850 5850 50  0001 C CNN
+F 3 "" H 2650 5500 50  0001 C CNN
+	1    2650 5500
+	1    0    0    -1
+$EndComp
+Wire Wire Line
+	3700 5600 3700 6250
 $EndSCHEMATC

Commit message: Edit PCB
Parts:
- added J10, J11, J12, J13, J8, J9: HEADER_1x01, Mlab_Pin_Headers:Straight_1x01, symbol MLAB_HEADER:HEADER_1x01
Connections:
- net GND: now also J13.1
- net PB4: now also J8.1; no longer R14.1
- net PB5: now also J9.1; no longer R16.1
- net PB6: now also J12.1; no longer R18.1
- net PB7: now also J11.1; no longer R17.1
- net SD_VDD: now also J10.1; no longer J1.4 (VDD)
Other:
- note added: "CD/DAT3"
- note added: "CLK"
- note added: "CMD"
- note added: "DAT0"
- moved on the sheet: C22, C25, J1, R14, R16, R17, R18

Commit message: Edit PCB
Connections:
- net PC3: now reaches U10.22 ((PCINT19/TMS)PC3)
- net PC3: now also J5.1
- net PC4: now reaches U10.23 ((PCINT20/TDO)PC4)
- net PC4: now also J4.1
- net PD2: no longer names the net of U10.11 ((PCINT26/RXD1/INT0)PD2)
- net PD2: no longer J5.1
- net PD3: no longer names the net of U10.12 ((PCINT27/TXD1/INT1)PD3)
- net PD3: no longer J4.1
Other:
- moved on the sheet: J4, J5
Changed lines of the file:
@@
 NoConn ~ 6850 4600
 NoConn ~ 6850 4000
-NoConn ~ 6850 3600
 NoConn ~ 6850 3900
 NoConn ~ 6850 3800
-NoConn ~ 6850 3700
 NoConn ~ 6850 2200
 NoConn ~ 6850 2100
@@
 NoConn ~ 6850 1800
 NoConn ~ 6850 1700
-Text Label 6950 4500 0    60   ~ 0
-PD3
-Text Label 6950 4400 0    60   ~ 0
-PD2
+Text Label 6950 3700 0    60   ~ 0
+PC4
+Text Label 6950 3600 0    60   ~ 0
+PC3
 $Comp
 L MLAB_HEADER:HEADER_1x01 J4
 U 1 1 5C6A22D0
-P 7400 4500
-F 0 "J4" H 7478 4505 60  0000 L CNN
-F 1 "HEADER_1x01" H 7478 4452 60  0001 L CNN
-F 2 "Mlab_Pin_Headers:Straight_1x01" H 7400 4500 60  0001 C CNN
-F 3 "" H 7400 4500 60  0000 C CNN
-	1    7400 4500
+P 7400 3700
+F 0 "J4" H 7478 3705 60  0000 L CNN
+F 1 "HEADER_1x01" H 7478 3652 60  0001 L CNN
+F 2 "Mlab_Pin_Headers:Straight_1x01" H 7400 3700 60  0001 C CNN
+F 3 "" H 7400 3700 60  0000 C CNN
+	1    7400 3700
 	1    0    0    -1
 $EndComp
@@
 L MLAB_HEADER:HEADER_1x01 J5
 U 1 1 5C6A319F
-P 7400 4400
-F 0 "J5" H 7478 4405 60  0000 L CNN
-F 1 "HEADER_1x01" H 7478 4352 60  0001 L CNN
-F 2 "Mlab_Pin_Headers:Straight_1x01" H 7400 4400 60  0001 C CNN
-F 3 "" H 7400 4400 60  0000 C CNN
-	1    7400 4400
+P 7400 3600
+F 0 "J5" H 7478 3605 60  0000 L CNN
+F 1 "HEADER_1x01" H 7478 3552 60  0001 L CNN
+F 2 "Mlab_Pin_Headers:Straight_1x01" H 7400 3600 60  0001 C CNN
+F 3 "" H 7400 3600 60  0000 C CNN
+	1    7400 3600
 	1    0    0    -1
 $EndComp
@@
 Wire Wire Line
 	6850 2400 6950 2400
-Wire Wire Line
-	6850 4400 7200 4400
-Wire Wire Line
-	6850 4500 7200 4500
 NoConn ~ 4850 1900
 NoConn ~ 4850 2300
@@
 Text Notes 1450 7050 0    60   ~ 0
 DAT0
+Wire Wire Line
+	6850 3600 7200 3600
+Wire Wire Line
+	6850 3700 7200 3700
+NoConn ~ 6850 4400
+NoConn ~ 6850 4500
 $EndSCHEMATC

Commit message: Edit
Parts:
- added C33: 10uF, Mlab_R:SMD-0805, symbol SPACEDOS02A_PCB01A-rescue:C-device-DATALOGGER01A-rescue-CCP2019V01A-rescue-SPAC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
- added C37: 100nF, Mlab_R:SMD-0805, symbol SPACEDOS02A_PCB01A-rescue:C-device-DATALOGGER01A-rescue-CCP2019V01A-rescue-SPAC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
- added J14, J15, J16, J17, J18, J20, J21, J23, J24, J25, J26, J27: HEADER_1x01, Mlab_Pin_Headers:Straight_1x01, symbol MLAB_HEADER:HEADER_1x01
- added J28: SD_Card-FPS009-4200-0, Mlab_CON:FPS009-4200-0, symbol MLAB_CONNECTORS:SD_Card-FPS009-4200-0
- added R24, R25, R26, R27: 100, Mlab_R:SMD-0805, symbol SPACEDOS02A_PCB01A-rescue:R-device-DATALOGGER01A-rescue-CCP2019V01A-rescue-SPAC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
- U11: UST_ID (none) -> 5c70984612875079b91f8a0c
- U6: UST_ID (none) -> 5c70984712875079b91f8b99
Connections:
- net GND: now also C33.2, C37.2, J20.1, J27.1, J28.12 (SHELL1), J28.3 (VSS), J28.6 (VSS)
- net SD_VDD: no longer C22.1, C25.1
- net at R14.1: now also J14.1
- net at R16.1: now also J15.1
- net at R17.1: now also J17.1
- net at R18.1: now also J18.1
- net SD_VDD2: now reaches J1.4 (VDD)
- net SD_VDD2: now also C22.1, C25.1, J16.1
- new net: J21.1, R24.1
- new net: J28.1 (CD/DAT3), R24.2
- new net: J23.1, R25.1
- new net: J28.2 (CMD), R25.2
- new net: J25.1, R26.1
- new net: J28.5 (CLK), R26.2
- new net: J26.1, R27.1
- new net: J28.7 (DAT0), R27.2
- new net SD_VDD3: C33.1, C37.1, J24.1, J28.4 (VDD)
Other:
- note removed: "CD/DAT3"
- note removed: "CLK"
- note removed: "CMD"
- note removed: "DAT0"
- moved on the sheet: J22

Commit message: Edit
Parts:
- C22, C33, C40: UST_ID (none) -> 5c70984812875079b91f8bbd
- C25, C26, C27, C28, C30, C31, C34, C35, C37, C39, C44, C47: UST_ID (none) -> 5c70984712875079b91f8b4c
- C43: UST_ID (none) -> 5c70984712875079b91f8b52
- J1: value SD_Card-Connector -> MCC-SD; UST_ID (none) -> 5c70984412875079b91f87f2
- J28: UST_ID (none) -> 5ccfe4d7128750448e45411b
- L1: UST_ID (none) -> 5c70984412875079b91f87ff
- R14, R16, R17, R18, R24, R25, R26, R27: UST_ID (none) -> 5c70984512875079b91f8977
- R20, R21, R23: UST_ID (none) -> 5c70984612875079b91f899f
- U10: UST_ID (none) -> 5c70984412875079b91f888e
- Y2: UST_ID (none) -> 5c70984712875079b91f8b1b
Changed lines of the file:
@@
 F 2 "Package_QFP:TQFP-44_10x10mm_P0.8mm" H 5850 3200 50  0001 C CIN
 F 3 "http://www.atmel.com/Images/Atmel-8272-8-bit-AVR-microcontroller-ATmega164A_PA-324A_PA-644A_PA-1284_P_datasheet.pdf" H 5850 3200 50  0001 C CNN
+F 4 "5c70984412875079b91f888e" H 5850 3200 50  0001 C CNN "UST_ID"
 	1    5850 3200
 	1    0    0    -1
@@
 F 2 "Mlab_R:SMD-0805" H 4188 2800 50  0001 C CNN
 F 3 "" H 4150 2950 50  0001 C CNN
+F 4 "5c70984812875079b91f8bbd" H 4150 2950 50  0001 C CNN "UST_ID"
 	1    4150 2950
 	1    0    0    -1
@@
 F 2 "Mlab_R:SMD-0805" H 4638 2800 50  0001 C CNN
 F 3 "" H 4600 2950 50  0001 C CNN
+F 4 "5c70984712875079b91f8b4c" H 4600 2950 50  0001 C CNN "UST_ID"
 	1    4600 2950
 	1    0    0    -1
@@
 F 2 "Mlab_R:SMD-0805" H 4438 1350 50  0001 C CNN
 F 3 "" H 4400 1500 50  0001 C CNN
+F 4 "5c70984712875079b91f8b52" H 4400 1500 50  0001 C CNN "UST_ID"
 	1    4400 1500
 	0    1    1    0
@@
 F 2 "Mlab_R:SMD-0805" V 4630 1200 50  0001 C CNN
 F 3 "" H 4700 1200 50  0001 C CNN
+F 4 "5c70984612875079b91f899f" H 4700 1200 50  0001 C CNN "UST_ID"
 	1    4700 1200
 	-1   0    0    1
@@
 F 2 "Mlab_R:SMD-0805" H 788 850 50  0001 C CNN
 F 3 "" H 750 1000 50  0001 C CNN
+F 4 "5c70984712875079b91f8b4c" H 750 1000 50  0001 C CNN "UST_ID"
 	1    750  1000
 	1    0    0    -1
@@
 F 2 "Mlab_R:SMD-0805" H 1238 850 50  0001 C CNN
 F 3 "" H 1200 1000 50  0001 C CNN
+F 4 "5c70984712875079b91f8b4c" H 1200 1000 50  0001 C CNN "UST_ID"
 	1    1200 1000
 	1    0    0    -1
@@
 F 2 "Mlab_R:SMD-0805" H 1688 850 50  0001 C CNN
 F 3 "" H 1650 1000 50  0001 C CNN
+F 4 "5c70984712875079b91f8b4c" H 1650 1000 50  0001 C CNN "UST_ID"
 	1    1650 1000
 	1    0    0    -1
@@
 F 2 "Mlab_R:SMD-1210" H 2100 800 50  0001 C CNN
 F 3 "" H 2100 800 50  0001 C CNN
+F 4 "5c70984412875079b91f87ff" H 2100 800 50  0001 C CNN "UST_ID"
 	1    2100 800
 	0    -1   -1   0
@@
 F 2 "Mlab_R:SMD-0805" H 2538 850 50  0001 C CNN
 F 3 "" H 2500 1000 50  0001 C CNN
+F 4 "5c70984712875079b91f8b4c" H 2500 1000 50  0001 C CNN "UST_ID"
 	1    2500 1000
 	1    0    0    -1
@@
 F 2 "Mlab_R:SMD-0805" V 630 3700 50  0001 C CNN
 F 3 "" H 700 3700 50  0001 C CNN
+F 4 "5c70984612875079b91f899f" H 700 3700 50  0001 C CNN "UST_ID"
 	1    700  3700
 	-1   0    0    1
@@
 F 2 "Mlab_R:SMD-0805" V 830 3700 50  0001 C CNN
 F 3 "" H 900 3700 50  0001 C CNN
+F 4 "5c70984612875079b91f899f" H 900 3700 50  0001 C CNN "UST_ID"
 	1    900  3700
 	-1   0    0    1
@@
 F 2 "Mlab_XTAL:ABS07" H 8750 4650 50  0001 C CNN
 F 3 "" H 8750 4650 50  0000 C CNN
+F 4 "5c70984712875079b91f8b1b" H 8750 4650 50  0001 C CNN "UST_ID"
 	1    8750 4650
 	1    0    0    -1
@@
 F 2 "Mlab_R:SMD-0805" H 10838 5700 50  0001 C CNN
 F 3 "" H 10800 5850 50  0001 C CNN
+F 4 "5c70984712875079b91f8b4c" H 10800 5850 50  0001 C CNN "UST_ID"
 	1    10800 5850
 	1    0    0    -1
@@
 F 2 "Mlab_R:SMD-0805" H 3138 850 50  0001 C CNN
 F 3 "" H 3100 1000 50  0001 C CNN
+F 4 "5c70984712875079b91f8b4c" H 3100 1000 50  0001 C CNN "UST_ID"
 	1    3100 1000
 	1    0    0    -1
@@
 F 2 "Mlab_R:SMD-0805" H 3588 850 50  0001 C CNN
 F 3 "" H 3550 1000 50  0001 C CNN
+F 4 "5c70984712875079b91f8b4c" H 3550 1000 50  0001 C CNN "UST_ID"
 	1    3550 1000
 	1    0    0    -1
@@
 F 2 "Mlab_R:SMD-0805" H 4088 850 50  0001 C CNN
 F 3 "" H 4050 1000 50  0001 C CNN
+F 4 "5c70984712875079b91f8b4c" H 4050 1000 50  0001 C CNN "UST_ID"
 	1    4050 1000
 	1    0    0    -1
@@
 F 2 "Mlab_R:SMD-0805" H 10538 2450 50  0001 C CNN
 F 3 "" H 10500 2600 50  0001 C CNN
+F 4 "5c70984712875079b91f8b4c" H 10500 2600 50  0001 C CNN "UST_ID"
 	1    10500 2600
 	1    0    0    -1
@@
 F 2 "Mlab_R:SMD-0805" H 4988 7100 50  0001 C CNN
 F 3 "" H 4950 7250 50  0001 C CNN
+F 4 "5c70984812875079b91f8bbd" H 4950 7250 50  0001 C CNN "UST_ID"
 	1    4950 7250
 	1    0    0    -1
@@
 F 2 "Mlab_R:SMD-0805" H 5438 7100 50  0001 C CNN
 F 3 "" H 5400 7250 50  0001 C CNN
+F 4 "5c70984712875079b91f8b4c" H 5400 7250 50  0001 C CNN "UST_ID"
 	1    5400 7250
 	1    0    0    -1
@@
 F 2 "Mlab_R:SMD-0805" V 2030 6400 50  0001 C CNN
 F 3 "" H 2100 6400 50  0001 C CNN
+F 4 "5c70984512875079b91f8977" H 2100 6400 50  0001 C CNN "UST_ID"
 	1    2100 6400
 	0    -1   -1   0
@@
 F 2 "Mlab_R:SMD-0805" V 2030 6500 50  0001 C CNN
 F 3 "" H 2100 6500 50  0001 C CNN
+F 4 "5c70984512875079b91f8977" H 2100 6500 50  0001 C CNN "UST_ID"
 	1    2100 6500
 	0    -1   -1   0
@@
 F 2 "Mlab_R:SMD-0805" V 2030 6800 50  0001 C CNN
 F 3 "" H 2100 6800 50  0001 C CNN
+F 4 "5c70984512875079b91f8977" H 2100 6800 50  0001 C CNN "UST_ID"
 	1    2100 6800
 	0    -1   -1   0
@@
 F 2 "Mlab_R:SMD-0805" V 2030 7000 50  0001 C CNN
 F 3 "" H 2100 7000 50  0001 C CNN
+F 4 "5c70984512875079b91f8977" H 2100 7000 50  0001 C CNN "UST_ID"
 	1    2100 7000
 	0    -1   -1   0
@@
 P 3500 6700
 F 0 "J1" H 3500 7365 50  0000 C CNN
-F 1 "SD_Card-Connector" H 3500 7274 50  0000 C CNN
+F 1 "MCC-SD" H 3500 7274 50  0000 C CNN
 F 2 "Mlab_CON:MCC-SD" H 3700 7050 50  0001 C CNN
 F 3 "" H 3500 6700 50  0001 C CNN
+F 4 "5c70984412875079b91f87f2" H 3500 6700 50  0001 C CNN "UST_ID"
 	1    3500 6700
 	1    0    0    -1
@@
 F 2 "Mlab_R:SMD-0805" H 4088 5350 50  0001 C CNN
 F 3 "" H 4050 5500 50  0001 C CNN
+F 4 "5c70984812875079b91f8bbd" H 4050 5500 50  0001 C CNN "UST_ID"
 	1    4050 5500
 	1    0    0    -1
@@
 F 2 "Mlab_R:SMD-0805" H 4538 5350 50  0001 C CNN
 F 3 "" H 4500 5500 50  0001 C CNN
+F 4 "5c70984712875079b91f8b4c" H 4500 5500 50  0001 C CNN "UST_ID"
 	1    4500 5500
 	1    0    0    -1
@@
 F 2 "Mlab_R:SMD-0805" V 1130 4650 50  0001 C CNN
 F 3 "" H 1200 4650 50  0001 C CNN
+F 4 "5c70984512875079b91f8977" H 1200 4650 50  0001 C CNN "UST_ID"
 	1    1200 4650
 	0    -1   -1   0
@@
 F 2 "Mlab_R:SMD-0805" V 1130 4750 50  0001 C CNN
 F 3 "" H 1200 4750 50  0001 C CNN
+F 4 "5c70984512875079b91f8977" H 1200 4750 50  0001 C CNN "UST_ID"
 	1    1200 4750
 	0    -1   -1   0
@@
 F 2 "Mlab_R:SMD-0805" V 1130 5050 50  0001 C CNN
 F 3 "" H 1200 5050 50  0001 C CNN
+F 4 "5c70984512875079b91f8977" H 1200 5050 50  0001 C CNN "UST_ID"
 	1    1200 5050
 	0    -1   -1   0
@@
 F 2 "Mlab_R:SMD-0805" V 1130 5250 50  0001 C CNN
 F 3 "" H 1200 5250 50  0001 C CNN
+F 4 "5c70984512875079b91f8977" H 1200 5250 50  0001 C CNN "UST_ID"
 	1    1200 5250
 	0    -1   -1   0
@@
 F 2 "Mlab_CON:FPS009-4200-0" H 2800 5300 50  0001 C CNN
 F 3 "" H 2600 4950 50  0001 C CNN
+F 4 "5ccfe4d7128750448e45411b" H 2600 4950 50  0001 C CNN "UST_ID"
 	1    2600 4950
 	1    0    0    -1
