File: hw/sch_pcb/SPACEDOS02A_PCB01A/power.sch (KiCad schematic (older format))
At the start: 16 parts, among them J1 HEADER_2x01, J2 HEADER_2x01_PARALLEL, J3 HEADER_2x01_PARALLEL, U8 TPS613222ADBV

Commit message: Edit
Parts:
- removed J1: HEADER_2x01, Mlab_Pin_Headers:Straight_1x02, symbol MLAB_HEADER:HEADER_2x01
Connections:
- no-connect marks 2 -> 0
Changed lines of the file:
@@
 	3850 2850 3850 3350
-$Comp
-L MLAB_HEADER:HEADER_2x01 J1
-U 1 1 5C82097F
-P 1600 2300
-F 0 "J1" H 1600 2441 60  0000 C CNN
-F 1 "HEADER_2x01" H 1600 2441 60  0001 C CNN
-F 2 "Mlab_Pin_Headers:Straight_1x02" H 1600 2300 60  0001 C CNN
-F 3 "" H 1600 2300 60  0000 C CNN
-	1    1600 2300
-	1    0    0    -1
-$EndComp
-NoConn ~ 1350 2300
-NoConn ~ 1850 2300
 $Comp
 L Device:Battery_Cell BT1

Commit message: Edit
Parts:
- BT1: footprint Mlab_Batery:BX0037 -> Mlab_Batery:BX0037_nez_sroubu
Changed lines of the file:
@@
 EESchema Schematic File Version 4
 LIBS:SPACEDOS02A_PCB01A-cache
-EELAYER 26 0
+EELAYER 29 0
 EELAYER END
 $Descr A4 11693 8268
@@
 F 0 "BT1" H 2218 3696 50  0000 L CNN
 F 1 "BX0037" H 2218 3605 50  0000 L CNN
-F 2 "Mlab_Batery:BX0037" V 2100 3660 50  0001 C CNN
+F 2 "Mlab_Batery:BX0037_nez_sroubu" V 2100 3660 50  0001 C CNN
 F 3 "~" V 2100 3660 50  0001 C CNN
 	1    2100 3600

Commit message: Edit
Parts:
- BT1: UST_ID (none) -> 5c70984412875079b91f87ed
- C29, C52: UST_ID (none) -> 5c70984412875079b91f880f
- C32, C54, C55: UST_ID (none) -> 5c70984712875079b91f8b4c
- C36, C42, C50: UST_ID (none) -> 5c70984812875079b91f8bbd
- D3: UST_ID (none) -> 5c70984512875079b91f88b2
- F2: value 2R2 -> 100mA; UST_ID (none) -> 5cc331a7128750448e54e8fa
- L3: UST_ID (none) -> 5cc3309d128750448e54e8d8
- U8: UST_ID (none) -> 5c7190ae1287500b4e112e04
Changed lines of the file:
@@
 F 2 "Resistor_SMD:R_0805_2012Metric_Pad1.15x1.40mm_HandSolder" H 6550 3300 50  0001 C CNN
 F 3 "~" H 6550 3300 50  0001 C CNN
+F 4 "5cc3309d128750448e54e8d8" H 6550 3300 50  0001 C CNN "UST_ID"
 	1    6550 3300
 	0    -1   -1   0
@@
 F 2 "Package_TO_SOT_SMD:SOT-23-5" H 7300 3400 60  0001 C CNN
 F 3 "" H 7300 3400 60  0001 C CNN
+F 4 "5c7190ae1287500b4e112e04" H 7300 3400 50  0001 C CNN "UST_ID"
 	1    7300 3400
 	1    0    0    -1
@@
 F 2 "Mlab_R:SMD-0805" H 7988 3400 50  0001 C CNN
 F 3 "" H 7950 3550 50  0001 C CNN
+F 4 "5c70984812875079b91f8bbd" H 7950 3550 50  0001 C CNN "UST_ID"
 	1    7950 3550
 	1    0    0    -1
@@
 F 2 "Mlab_R:SMD-0805" H 8438 3400 50  0001 C CNN
 F 3 "" H 8400 3550 50  0001 C CNN
+F 4 "5c70984812875079b91f8bbd" H 8400 3550 50  0001 C CNN "UST_ID"
 	1    8400 3550
 	1    0    0    -1
@@
 F 2 "Mlab_R:SMD-0805" H 6238 3400 50  0001 C CNN
 F 3 "" H 6200 3550 50  0001 C CNN
+F 4 "5c70984712875079b91f8b4c" H 6200 3550 50  0001 C CNN "UST_ID"
 	1    6200 3550
 	1    0    0    -1
@@
 F 2 "Mlab_L:FIR_0805" V 8950 3400 50  0001 C CNN
 F 3 "http://www.murata.com/~/media/webrenewal/support/library/catalog/products/emc/emifil/c31e.ashx?la=en-gb" V 8950 3400 50  0001 C CNN
+F 4 "5c70984412875079b91f880f" H 8950 3400 50  0001 C CNN "UST_ID"
 	1    8950 3400
 	1    0    0    -1
@@
 F 2 "Mlab_R:SMD-0805" H 9388 3350 50  0001 C CNN
 F 3 "" H 9350 3500 50  0001 C CNN
+F 4 "5c70984712875079b91f8b4c" H 9350 3500 50  0001 C CNN "UST_ID"
 	1    9350 3500
 	1    0    0    -1
@@
 F 2 "Diode_SMD:D_MiniMELF" H 2800 3550 50  0001 C CNN
 F 3 "" H 2800 3550 50  0001 C CNN
+F 4 "5c70984512875079b91f88b2" H 2800 3550 50  0001 C CNN "UST_ID"
 	1    2800 3550
 	0    1    1    0
@@
 F 2 "Mlab_L:FIR_0805" V 3450 3450 50  0001 C CNN
 F 3 "http://www.murata.com/~/media/webrenewal/support/library/catalog/products/emc/emifil/c31e.ashx?la=en-gb" V 3450 3450 50  0001 C CNN
+F 4 "5c70984412875079b91f880f" H 3450 3450 50  0001 C CNN "UST_ID"
 	1    3450 3450
 	1    0    0    -1
@@
 F 2 "Mlab_R:SMD-0805" H 3888 3400 50  0001 C CNN
 F 3 "" H 3850 3550 50  0001 C CNN
+F 4 "5c70984712875079b91f8b4c" H 3850 3550 50  0001 C CNN "UST_ID"
 	1    3850 3550
 	1    0    0    -1
@@
 Wire Wire Line
 	3450 3550 3450 3750
-$Comp
-L SPACEDOS02A_PCB01A-rescue:Polyfuse-device-DATALOGGER01A-rescue-CCP2019V01A-rescue-SPACEDOS01A_PCB01A-rescue-SPACEDOS01B_PCB01A-rescue-SPACEDOS01B_PCB01A-rescue F?
-U 1 1 5C58939A
-P 2450 3350
-AR Path="/5C4AEDD8/5C58939A" Ref="F?"  Part="1"
-AR Path="/5C69BCB4/5C58939A" Ref="F2"  Part="1"
-F 0 "F2" V 2225 3350 50  0000 C CNN
-F 1 "2R2" V 2300 3350 50  0000 C CNN
-F 2 "Mlab_R:SMD-0805" H 2500 3150 50  0001 L CNN
-F 3 "" H 2450 3350 50  0001 C CNN
-	1    2450 3350
-	0    1    1    0
-$EndComp
 Wire Wire Line
 	2600 3350 2800 3350
@@
 F 2 "Mlab_R:SMD-0805" H 3138 3400 50  0001 C CNN
 F 3 "" H 3100 3550 50  0001 C CNN
+F 4 "5c70984812875079b91f8bbd" H 3100 3550 50  0001 C CNN "UST_ID"
 	1    3100 3550
 	1    0    0    -1
@@
 F 2 "Mlab_Batery:BX0037_nez_sroubu" V 2100 3660 50  0001 C CNN
 F 3 "~" V 2100 3660 50  0001 C CNN
+F 4 "5c70984412875079b91f87ed" H 2100 3600 50  0001 C CNN "UST_ID"
 	1    2100 3600
 	1    0    0    -1
@@
 Wire Wire Line
 	2100 3700 2100 3750
+$Comp
+L SPACEDOS02A_PCB01A-rescue:Polyfuse-device-DATALOGGER01A-rescue-CCP2019V01A-rescue-SPACEDOS01A_PCB01A-rescue-SPACEDOS01B_PCB01A-rescue-SPACEDOS01B_PCB01A-rescue F?
+U 1 1 5C58939A
+P 2450 3350
+AR Path="/5C4AEDD8/5C58939A" Ref="F?"  Part="1"
+AR Path="/5C69BCB4/5C58939A" Ref="F2"  Part="1"
+F 0 "F2" V 2225 3350 50  0000 C CNN
+F 1 "100mA" V 2300 3350 50  0000 C CNN
+F 2 "Mlab_R:SMD-0805" H 2500 3150 50  0001 L CNN
+F 3 "" H 2450 3350 50  0001 C CNN
+F 4 "5cc331a7128750448e54e8fa" H 2450 3350 50  0001 C CNN "UST_ID"
+	1    2450 3350
+	0    1    1    0
+$EndComp
 $EndSCHEMATC
