File: hw/sch_pcb/SPACEDOS02B_PCB01A/SPACEDOS02B_PCB01A.kicad_sch (KiCad schematic)
At the start: 47 parts, among them M6 BMI-S-210-F, M8 BMI-S-210-F, U1 OPA2314, U2 OPA2314, U3 ISL21080DIH312Z-TK 1V25, U4 TS7211, U5 TS5A4594

Commit message: Add new submodule with UST titleblock.
Other:
- company: Mlab www.mlab.cz -> Universal Scientific  \n Technologies s.r.o.
- title: NAME -> SPACEDOS02B

Commit message: Oprava otvíratelnosti schéma.
Other:
- company: Universal Scientific  \n Technologies s.r.o. -> Mlab www.mlab.cz
- title: SPACEDOS02B -> NAME

Commit message: Edit schema
Connections:
- net +3V3 renamed POWER_ANALOG_3V3
Changed lines of the file:
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@@
-    (stroke (width 0) (type default) (color 0 0 0 0))
-  )
-  (wire (pts (xy 25.4 22.86) (xy 25.4 24.13))
-    (stroke (width 0) (type default) (color 0 0 0 0))
-  )
-  (wire (pts (xy 25.4 24.13) (xy 35.56 24.13))
     (stroke (width 0) (type default) (color 0 0 0 0))
   )
@@
   )
   (wire (pts (xy 34.29 182.88) (xy 34.29 181.61))
+    (stroke (width 0) (type default) (color 0 0 0 0))
+  )
+  (wire (pts (xy 35.56 24.13) (xy 34.29 24.13))
     (stroke (width 0) (type default) (color 0 0 0 0))
   )
@@
   (label "A/D" (at 269.24 96.52 90)
     (effects (font (size 1.524 1.524)) (justify left bottom))
+  )
+  (global_label "POWER_ANALOG_3V3" (shape input) (at 34.29 24.13 180) (fields_autoplaced)
+    (effects (font (size 1.524 1.524)) (justify right))
+    (property "Intersheet References" "${INTERSHEET_REFS}" (id 0) (at 8.6411 24.0348 0)
+      (effects (font (size 1.524 1.524)) (justify right) hide)
+    )
+  )
+  (global_label "POWER_ANALOG_3V3" (shape input) (at 114.3 30.48 90) (fields_autoplaced)
+    (effects (font (size 1.524 1.524)) (justify left))
+    (property "Intersheet References" "${INTERSHEET_REFS}" (id 0) (at 114.3952 4.8311 90)
+      (effects (font (size 1.524 1.524)) (justify left) hide)
+    )
   )
   (global_label "PB0" (shape input) (at 267.97 130.81 0) (fields_autoplaced)
@@
     )
     (property "Datasheet" "" (id 3) (at 24.13 171.45 0)
-      (effects (font (size 1.27 1.27)) hide)
-    )
-    (pin "1")
-  )
-  (symbol (lib_id "power:+3.3V") (at 25.4 22.86 0) (unit 1)
-    (in_bom yes) (on_board yes)
-    (property "Reference" "#PWR0106" (id 0) (at 25.4 26.67 0)
-      (effects (font (size 1.27 1.27)) hide)
-    )
-    (property "Value" "+3.3V" (id 1) (at 25.781 18.4658 0))
-    (property "Footprint" "" (id 2) (at 25.4 22.86 0)
-      (effects (font (size 1.27 1.27)) hide)
-    )
-    (property "Datasheet" "" (id 3) (at 25.4 22.86 0)
-      (effects (font (size 1.27 1.27)) hide)
-    )
-    (pin "1")
-  )
-  (symbol (lib_id "power:+3.3V") (at 114.3 30.48 0) (unit 1)
-    (in_bom yes) (on_board yes)
-    (property "Reference" "#PWR0107" (id 0) (at 114.3 34.29 0)
-      (effects (font (size 1.27 1.27)) hide)
-    )
-    (property "Value" "+3.3V" (id 1) (at 114.681 26.0858 0))
-    (property "Footprint" "" (id 2) (at 114.3 30.48 0)
-      (effects (font (size 1.27 1.27)) hide)
-    )
-    (property "Datasheet" "" (id 3) (at 114.3 30.48 0)
       (effects (font (size 1.27 1.27)) hide)
     )
@@
       (reference "#PWR0105") (unit 1) (value "GND") (footprint "")
     )
-    (path "/00000000-0000-0000-0000-00005c6997a5"
-      (reference "#PWR0106") (unit 1) (value "+3.3V") (footprint "")
-    )
-    (path "/00000000-0000-0000-0000-00005c699bf2"
-      (reference "#PWR0107") (unit 1) (value "+3.3V") (footprint "")
-    )
     (path "/00000000-0000-0000-0000-00005c4aedd8/00000000-0000-0000-0000-00005c634bea"
       (reference "#PWR0108") (unit 1) (value "+3.3V") (footprint "")
@@
       (reference "#PWR0125") (unit 1) (value "+3.3V") (footprint "")
     )
-    (path "/00000000-0000-0000-0000-00005c4aedd8/d731d43a-eac4-4e7c-88b1-e99132222286"
-      (reference "#PWR0126") (unit 1) (value "+5V") (footprint "")
-    )
     (path "/00000000-0000-0000-0000-00005c4aedd8/c105aa78-22fa-412d-a9a2-0a21aa50cf12"
       (reference "#PWR0127") (unit 1) (value "GND") (footprint "")
@@
       (reference "#PWR0158") (unit 1) (value "GND") (footprint "")
     )
-    (path "/00000000-0000-0000-0000-00005c69bcb4/00000000-0000-0000-0000-00005c6d0ec0"
-      (reference "#PWR0161") (unit 1) (value "VDD") (footprint "")
-    )
     (path "/00000000-0000-0000-0000-00005c69bcb4/00000000-0000-0000-0000-00005c6d0ec8"
       (reference "#PWR0163") (unit 1) (value "GND") (footprint "")
@@
       (reference "#PWR0174") (unit 1) (value "VDD") (footprint "")
     )
+    (path "/00000000-0000-0000-0000-00005c69bcb4/13f5e65a-bc3e-44e6-9299-9163c7f13f78"
+      (reference "#PWR?") (unit 1) (value "GND") (footprint "")
+    )
+    (path "/00000000-0000-0000-0000-00005c69bcb4/7aa5f446-b73d-4976-97b6-35d0fab45f42"
+      (reference "#PWR?") (unit 1) (value "GND") (footprint "")
+    )
+    (path "/00000000-0000-0000-0000-00005c69bcb4/a3a3b2cd-d10b-4600-9ee2-29a111b3bec7"
+      (reference "#PWR?") (unit 1) (value "GND") (footprint "")
+    )
     (path "/00000000-0000-0000-0000-00005c69bcb4/00000000-0000-0000-0000-00005cc376a8"
       (reference "BT1") (unit 1) (value "BX0037") (footprint "Mlab_Batery:BX0037_nez_sroubu")
@@
       (reference "C55") (unit 1) (value "100nF") (footprint "Mlab_R:SMD-0805")
     )
+    (path "/00000000-0000-0000-0000-00005c69bcb4/07fd7f88-d3ee-4c7f-8871-56d908141d09"
+      (reference "C?") (unit 1) (value "10uF") (footprint "Mlab_R:SMD-0805")
+    )
+    (path "/00000000-0000-0000-0000-00005c69bcb4/2df070f1-98d9-42aa-bbea-aa9f4064b7be"
+      (reference "C?") (unit 1) (value "1uF") (footprint "Mlab_R:SMD-0603")
+    )
+    (path "/00000000-0000-0000-0000-00005c69bcb4/757d3c7b-0129-4776-97ce-a5ec06b9ac70"
+      (reference "C?") (unit 1) (value "100nF") (footprint "Mlab_R:SMD-0603")
+    )
     (path "/00000000-0000-0000-0000-00005c80a3e9"
       (reference "D1") (unit 1) (value "S2744-09") (footprint "Mlab_D:HAMAMATSU_S2744-09")
@@
       (reference "L3") (unit 1) (value "DFE252012P-4R7M") (footprint "Resistor_SMD:R_0805_2012Metric_Pad1.15x1.40mm_HandSolder")
     )
+    (path "/00000000-0000-0000-0000-00005c4aedd8/0293d1f7-b050-4324-afda-8e53bf70b6fd"
+      (reference "L?") (unit 1) (value "L") (footprint "")
+    )
     (path "/00000000-0000-0000-0000-00005b47dba2"
       (reference "M6") (unit 1) (value "BMI-S-210-F") (footprint "Mlab_Mechanical:BMI-S-210-F")
@@
       (reference "U11") (unit 1) (value "PCF85263A") (footprint "Mlab_IO:TSSOP-10_3x3mm_Pitch0.5mm")
     )
+    (path "/00000000-0000-0000-0000-00005c69bcb4/9026c369-5914-4d03-a792-0a84a97d77cc"
+      (reference "U?") (unit 1) (value "MIC5504-3.3YM5") (footprint "Package_TO_SOT_SMD:SOT-23-5")
+    )
     (path "/00000000-0000-0000-0000-00005c4aedd8/dd3d6d5f-51af-4a06-b57d-aea9895cf705"

Commit message: Clean repository
Other:
- company: Mlab www.mlab.cz -> UST
- title: NAME -> (none)
