File: hw/sch_pcb/SPACEDOS02B_PCB01A/cpu.kicad_sch (KiCad schematic)
At the start: 58 parts, among them J1 MCC-SD, J10 HEADER_1x01, J11 HEADER_1x01, J12 HEADER_1x01, J13 HEADER_1x01, J14 HEADER_1x01, J15 HEADER_1x01, J16 HEADER_1x01, J17 HEADER_1x01, J18 HEADER_1x01, J19 HEADER_2x01_PARALLEL, J20 HEADER_1x01, J21 HEADER_1x01, J22 HEADER_2x03, J23 HEADER_1x01, J24 HEADER_1x01, J25 HEADER_1x01, J26 HEADER_1x01, J27 HEADER_1x01, J28 SD_Card-FPS009-4200-0, J4 HEADER_1x01, J5 HEADER_1x01, J6 HEADER_1x01, J7 HEADER_1x01, J8 HEADER_1x01, J9 HEADER_1x01, U10 ATMEGA1284P-AU, U11 PCF85263A, U6 AT24CS64-SSHM, Y2 ABS07-120-32.768KHZ-T

Commit message: Oprava otvíratelnosti schéma.
Parts:
- added U7: IR4302, Package_DFN_QFN:Infineon_PQFN-44-31-5EP_7x7mm_P0.5mm, symbol Amplifier_Audio:IR4302
Connections:
- new net: U7.15 (COM), U7.28 (COM), U7.31 (COM)
- new net: U7.18 (VS1), U7.20 (VS1)

Commit message: #4 add crystal
Parts:
- removed U7: IR4302, Package_DFN_QFN:Infineon_PQFN-44-31-5EP_7x7mm_P0.5mm, symbol Amplifier_Audio:IR4302
- added C38, C41: 15pF, Mlab_R:SMD-0805, symbol Device:C
- added Y1: 1,8432MHz, Crystal:Crystal_HC49-U_Horizontal, symbol Device:Crystal_Small
Connections:
- net GND: now also C38.2, C41.2
- net at U10.7 (XTAL2): now also C38.1, Y1.1
- net at U10.8 (XTAL1): now also C41.1, Y1.2
- no-connect marks 21 -> 19
Changed lines of the file:
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@@
   (junction (at 63.5 181.61) (diameter 0) (color 0 0 0 0))
   (junction (at 109.22 133.35) (diameter 0) (color 0 0 0 0))
+  (junction (at 111.76 48.26) (diameter 0) (color 0 0 0 0))
+  (junction (at 111.76 58.42) (diameter 0) (color 0 0 0 0))
   (junction (at 116.84 68.58) (diameter 0) (color 0 0 0 0))
   (junction (at 119.38 38.1) (diameter 0) (color 0 0 0 0))
@@
   (junction (at 227.33 63.5) (diameter 0) (color 0 0 0 0))
   (junction (at 227.33 66.04) (diameter 0) (color 0 0 0 0))
-  (no_connect (at 123.19 48.26))
-  (no_connect (at 123.19 58.42))
   (no_connect (at 173.99 43.18))
   (no_connect (at 173.99 45.72))
@@
     (stroke (width 0) (type default) (color 0 0 0 0))
   )
+  (wire (pts (xy 92.71 48.26) (xy 95.25 48.26))
+    (stroke (width 0) (type default) (color 0 0 0 0))
+  )
+  (wire (pts (xy 92.71 58.42) (xy 95.25 58.42))
+    (stroke (width 0) (type default) (color 0 0 0 0))
+  )
   (wire (pts (xy 92.71 128.27) (xy 92.71 144.78))
     (stroke (width 0) (type default) (color 0 0 0 0))
@@
     (stroke (width 0) (type default) (color 0 0 0 0))
   )
+  (wire (pts (xy 102.87 48.26) (xy 111.76 48.26))
+    (stroke (width 0) (type default) (color 0 0 0 0))
+  )
+  (wire (pts (xy 102.87 58.42) (xy 111.76 58.42))
+    (stroke (width 0) (type default) (color 0 0 0 0))
+  )
   (wire (pts (xy 102.87 133.35) (xy 102.87 135.89))
     (stroke (width 0) (type default) (color 0 0 0 0))
@@
     (stroke (width 0) (type default) (color 0 0 0 0))
   )
+  (wire (pts (xy 111.76 48.26) (xy 111.76 50.8))
+    (stroke (width 0) (type default) (color 0 0 0 0))
+  )
+  (wire (pts (xy 111.76 58.42) (xy 111.76 55.88))
+    (stroke (width 0) (type default) (color 0 0 0 0))
+  )
   (wire (pts (xy 111.76 172.72) (xy 115.57 172.72))
     (stroke (width 0) (type default) (color 0 0 0 0))
@@
   )
   (wire (pts (xy 119.38 38.1) (xy 123.19 38.1))
+    (stroke (width 0) (type default) (color 0 0 0 0))
+  )
+  (wire (pts (xy 123.19 48.26) (xy 111.76 48.26))
+    (stroke (width 0) (type default) (color 0 0 0 0))
+  )
+  (wire (pts (xy 123.19 58.42) (xy 111.76 58.42))
     (stroke (width 0) (type default) (color 0 0 0 0))
   )
@@
     (pin "1")
   )
+  (symbol (lib_id "power:GND") (at 92.71 48.26 270) (unit 1)
+    (in_bom yes) (on_board yes)
+    (property "Reference" "#PWR0155" (id 0) (at 86.36 48.26 0)
+      (effects (font (size 1.27 1.27)) hide)
+    )
+    (property "Value" "GND" (id 1) (at 88.3158 48.387 0))
+    (property "Footprint" "" (id 2) (at 92.71 48.26 0)
+      (effects (font (size 1.27 1.27)) hide)
+    )
+    (property "Datasheet" "" (id 3) (at 92.71 48.26 0)
+      (effects (font (size 1.27 1.27)) hide)
+    )
+    (pin "1")
+  )
+  (symbol (lib_id "power:GND") (at 92.71 58.42 270) (unit 1)
+    (in_bom yes) (on_board yes)
+    (property "Reference" "#PWR0151" (id 0) (at 86.36 58.42 0)
+      (effects (font (size 1.27 1.27)) hide)
+    )
+    (property "Value" "GND" (id 1) (at 88.3158 58.547 0))
+    (property "Footprint" "" (id 2) (at 92.71 58.42 0)
+      (effects (font (size 1.27 1.27)) hide)
+    )
+    (property "Datasheet" "" (id 3) (at 92.71 58.42 0)
+      (effects (font (size 1.27 1.27)) hide)
+    )
+    (pin "1")
+  )
   (symbol (lib_id "power:GND") (at 92.71 144.78 0) (unit 1)
     (in_bom yes) (on_board yes)
@@
     (pin "2")
   )
+  (symbol (lib_id "Device:Crystal_Small") (at 111.76 53.34 270) (unit 1)
+    (in_bom yes) (on_board yes) (fields_autoplaced)
+    (property "Reference" "Y1" (id 0) (at 113.9191 52.4315 90)
+      (effects (font (size 1.27 1.27)) (justify left))
+    )
+    (property "Value" "1,8432MHz" (id 1) (at 113.9191 55.2066 90)
+      (effects (font (size 1.27 1.27)) (justify left))
+    )
+    (property "Footprint" "Crystal:Crystal_HC49-U_Horizontal" (id 2) (at 111.76 53.34 0)
+      (effects (font (size 1.27 1.27)) hide)
+    )
+    (property "Datasheet" "1.8432M-HC49 YIC" (id 3) (at 111.76 53.34 0)
+      (effects (font (size 1.27 1.27)) hide)
+    )
+    (pin "1")
+    (pin "2")
+  )
   (symbol (lib_id "MLAB_HEADER:HEADER_1x01") (at 20.32 118.11 180) (unit 1)
     (in_bom yes) (on_board yes)
@@
     )
     (property "UST_ID" "5c70984712875079b91f8b4c" (id 4) (at 90.17 25.4 0)
+      (effects (font (size 1.27 1.27)) hide)
+    )
+    (pin "1")
+    (pin "2")
+  )
+  (symbol (lib_id "Device:C") (at 99.06 48.26 270) (unit 1)
+    (in_bom yes) (on_board yes)
+    (property "Reference" "C38" (id 0) (at 99.06 44.6744 90))
+    (property "Value" "15pF" (id 1) (at 99.06 52.5295 90))
+    (property "Footprint" "Mlab_R:SMD-0805" (id 2) (at 95.25 49.2252 0)
+      (effects (font (size 1.27 1.27)) hide)
+    )
+    (property "Datasheet" "~" (id 3) (at 99.06 48.26 0)
+      (effects (font (size 1.27 1.27)) hide)
+    )
+    (pin "1")
+    (pin "2")
+  )
+  (symbol (lib_id "Device:C") (at 99.06 58.42 270) (unit 1)
+    (in_bom yes) (on_board yes)
+    (property "Reference" "C41" (id 0) (at 99.06 54.8344 90))
+    (property "Value" "15pF" (id 1) (at 99.06 62.6895 90))
+    (property "Footprint" "Mlab_R:SMD-0805" (id 2) (at 95.25 59.3852 0)
+      (effects (font (size 1.27 1.27)) hide)
+    )
+    (property "Datasheet" "~" (id 3) (at 99.06 58.42 0)
       (effects (font (size 1.27 1.27)) hide)
     )
@@
     (pin "8")
   )
-  (symbol (lib_id "Amplifier_Audio:IR4302") (at 208.28 46.99 0) (unit 1)
-    (in_bom yes) (on_board yes) (fields_autoplaced)
-    (property "Reference" "U7" (id 0) (at 208.28 22.8304 0))
-    (property "Value" "IR4302" (id 1) (at 208.28 25.6055 0))
-    (property "Footprint" "Package_DFN_QFN:Infineon_PQFN-44-31-5EP_7x7mm_P0.5mm" (id 2) (at 208.28 46.99 0)
-      (effects (font (size 1.27 1.27) italic) hide)
-    )
-    (property "Datasheet" "https://www.infineon.com/dgdl/ir4302.pdf?fileId=5546d462533600a4015355d602a9181d" (id 3) (at 208.28 46.99 0)
-      (effects (font (size 1.27 1.27)) hide)
-    )
-    (pin "1")
-    (pin "10")
-    (pin "11")
-    (pin "12")
-    (pin "13")
-    (pin "14")
-    (pin "15")
-    (pin "16")
-    (pin "17")
-    (pin "18")
-    (pin "19")
-    (pin "20")
-    (pin "21")
-    (pin "28")
-    (pin "29")
-    (pin "30")
-    (pin "31")
-    (pin "5")
-    (pin "6")
-    (pin "7")
-    (pin "8")
-    (pin "9")
-  )
   (symbol (lib_id "MLAB_CONNECTORS:SD_Card-FPS009-4200-0") (at 66.04 125.73 0) (unit 1)

Commit message: Edit PCB
Parts:
- removed C22, C33: 10uF, Mlab_R:SMD-0805, symbol SPACEDOS02A_PCB01A-rescue:C-device-DATALOGGER01A-rescue-CCP2019V01A-rescue-SPAC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
- removed C25, C37: 100nF, Mlab_R:SMD-0805, symbol SPACEDOS02A_PCB01A-rescue:C-device-DATALOGGER01A-rescue-CCP2019V01A-rescue-SPAC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
- removed J1: MCC-SD, Mlab_CON:MCC-SD, symbol MLAB_CONNECTORS:SD_Card-Connector
- removed J14, J15, J16, J17, J18, J20, J21, J23, J24, J25, J26, J27: HEADER_1x01, Mlab_Pin_Headers:Straight_1x01, symbol MLAB_HEADER:HEADER_1x01
- removed J28: SD_Card-FPS009-4200-0, Mlab_CON:FPS009-4200-0, symbol MLAB_CONNECTORS:SD_Card-FPS009-4200-0
- removed R14, R16, R17, R18, R24, R25, R26, R27: 100, Mlab_R:SMD-0805, symbol SPACEDOS02A_PCB01A-rescue:R-device-DATALOGGER01A-rescue-CCP2019V01A-rescue-SPAC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
Other:
- note added: "FOR SD CARD PCB"

Commit message: Edit schema
Parts:
- added J1: SM08B-GHS-TB, Connector_JST:JST_GH_SM08B-GHS-TB_1x08-1MP_P1.25mm_Horizontal, symbol MLAB_CONNECTORS_JST:SM08B-GHS-TB
- added J14: SM06B-GHS-TB, Connector_JST:JST_GH_SM06B-GHS-TB_1x06-1MP_P1.25mm_Horizontal, symbol MLAB_CONNECTORS_JST:SM06B-GHS-TB
- added R14, R16: 100R, Resistor_SMD:R_0603_1608Metric, symbol SHT31V01A-rescue:R
- added R17, R18: 33R, Resistor_SMD:R_0603_1608Metric, symbol Device:R
Connections:
- net GND: now also J1.8, J1.MP, J14.6, J14.MP
- net PC0: now also R16.1
- net PC1: now also R14.1
- net RX0: now also R17.1
- net TX0: now also R18.1
- new net: J1.4, R14.2
- new net: J1.5, R16.2
- new net: J14.3, R18.2
- new net: J14.2, R17.2
- new net +5V: J14.1
- new net EXTINT: J1.2
- new net GEO_STAT: J1.3
- new net RX1: J1.7
- new net TIMEPULSE: J1.1
- new net TX1: J1.6
- no-connect marks 19 -> 21

Commit message: Edit
Parts:
- removed R14, R16: 100R, Resistor_SMD:R_0603_1608Metric, symbol SHT31V01A-rescue:R
- removed R17, R18: 33R, Resistor_SMD:R_0603_1608Metric, symbol Device:R
Connections:
- net EXTINT: now also U10.14 ((PCINT294/OC1A)PD5)
- net GEO_STAT: now also U10.15 ((PCINT30/OC2B/ICP)PD6)
- net PC0: now also J1.5
- net PC1: now also J1.4
- net RX0: now also J14.2
- net RX1: now also U10.11 ((PCINT26/RXD1/INT0)PD2)
- net TIMEPULSE: now also U10.13 ((PCINT28/XCK1/OC1B)PD4)
- net TX0: now also J14.3
- net TX1: now also U10.12 ((PCINT27/TXD1/INT1)PD3)
- no-connect marks 21 -> 16
Changed lines of the file:
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@@
   (no_connect (at 173.99 99.06))
   (no_connect (at 173.99 101.6))
-  (no_connect (at 173.99 111.76))
-  (no_connect (at 173.99 114.3))
-  (no_connect (at 173.99 116.84))
-  (no_connect (at 173.99 119.38))
-  (no_connect (at 173.99 121.92))
   (no_connect (at 173.99 124.46))
   (no_connect (at 261.62 133.35))
@@
     (stroke (width 0) (type default) (color 0 0 0 0))
   )
-  (wire (pts (xy 66.04 171.45) (xy 68.58 171.45))
-    (stroke (width 0) (type solid) (color 0 0 0 0))
-  )
-  (wire (pts (xy 66.04 173.99) (xy 68.58 173.99))
-    (stroke (width 0) (type solid) (color 0 0 0 0))
-  )
   (wire (pts (xy 76.2 171.45) (xy 86.995 171.45))
     (stroke (width 0) (type solid) (color 0 0 0 0))
@@
     (stroke (width 0) (type default) (color 0 0 0 0))
   )
-  (wire (pts (xy 102.87 168.91) (xy 107.95 168.91))
-    (stroke (width 0) (type solid) (color 0 0 0 0))
-  )
-  (wire (pts (xy 102.87 171.45) (xy 107.95 171.45))
-    (stroke (width 0) (type solid) (color 0 0 0 0))
-  )
   (wire (pts (xy 105.41 68.58) (xy 105.41 71.12))
     (stroke (width 0) (type default) (color 0 0 0 0))
@@
     (stroke (width 0) (type default) (color 0 0 0 0))
   )
+  (wire (pts (xy 173.99 111.76) (xy 176.53 111.76))
+    (stroke (width 0) (type default) (color 0 0 0 0))
+  )
+  (wire (pts (xy 173.99 119.38) (xy 176.53 119.38))
+    (stroke (width 0) (type default) (color 0 0 0 0))
+  )
+  (wire (pts (xy 173.99 121.92) (xy 176.53 121.92))
+    (stroke (width 0) (type default) (color 0 0 0 0))
+  )
   (wire (pts (xy 176.53 63.5) (xy 176.53 66.04))
     (stroke (width 0) (type default) (color 0 0 0 0))
@@
     (stroke (width 0) (type default) (color 0 0 0 0))
   )
+  (wire (pts (xy 176.53 114.3) (xy 173.99 114.3))
+    (stroke (width 0) (type default) (color 0 0 0 0))
+  )
+  (wire (pts (xy 176.53 116.84) (xy 173.99 116.84))
+    (stroke (width 0) (type default) (color 0 0 0 0))
+  )
   (wire (pts (xy 194.31 144.78) (xy 200.66 144.78))
     (stroke (width 0) (type default) (color 0 0 0 0))
@@
     (effects (font (size 1.524 1.524)) (justify left bottom))
   )
-  (label "PC1" (at 66.04 171.45 180)
+  (label "PC1" (at 76.2 171.45 180)
     (effects (font (size 1.524 1.524)) (justify right bottom))
   )
-  (label "PC0" (at 66.04 173.99 180)
+  (label "PC0" (at 76.2 173.99 180)
     (effects (font (size 1.524 1.524)) (justify right bottom))
   )
@@
     (effects (font (size 1.524 1.524)) (justify left bottom))
   )
-  (label "RX0" (at 102.87 168.91 0)
-    (effects (font (size 1.524 1.524)) (justify left bottom))
-  )
-  (label "TX0" (at 102.87 171.45 0)
-    (effects (font (size 1.524 1.524)) (justify left bottom))
+  (label "RX0" (at 115.57 168.91 180)
+    (effects (font (size 1.524 1.524)) (justify right bottom))
+  )
+  (label "TX0" (at 115.57 171.45 180)
+    (effects (font (size 1.524 1.524)) (justify right bottom))
   )
   (label "RST#_P" (at 116.84 38.1 90)
@@
   (label "TX0" (at 176.53 109.22 0)
     (effects (font (size 1.524 1.524)) (justify left bottom))
+  )
+  (label "RX1" (at 176.53 111.76 0)
+    (effects (font (size 1.524 1.524)) (justify left bottom))
+  )
+  (label "TX1" (at 176.53 114.3 0)
+    (effects (font (size 1.524 1.524)) (justify left bottom))
+  )
+  (label "TIMEPULSE" (at 176.53 116.84 0)
+    (effects (font (size 1.524 1.524)) (justify left bottom))
+  )
+  (label "EXTINT" (at 176.53 119.38 0)
+    (effects (font (size 1.27 1.27)) (justify left bottom))
+  )
+  (label "GEO_STAT" (at 176.53 121.92 0)
+    (effects (font (size 1.27 1.27)) (justify left bottom))
   )
   (label "SD_VDD" (at 179.07 66.04 0)
@@
       (effects (font (size 1.27 1.27)) hide)
     )
-    (pin "1")
-    (pin "2")
-  )
-  (symbol (lib_id "SHT31V01A-rescue:R") (at 72.39 171.45 90) (unit 1)
-    (in_bom yes) (on_board yes)
-    (property "Reference" "R14" (id 0) (at 72.39 169.418 90))
-    (property "Value" "100R" (id 1) (at 72.39 171.45 90))
-    (property "Footprint" "Resistor_SMD:R_0603_1608Metric" (id 2) (at 72.39 173.228 90)
-      (effects (font (size 1.27 1.27)) hide)
-    )
-    (property "Datasheet" "" (id 3) (at 72.39 171.45 0))
-    (property "UST_ID" "5c70984512875079b91f8956" (id 4) (at 72.39 171.45 0)
-      (effects (font (size 1.27 1.27)) hide)
-    )
-    (pin "1")
-    (pin "2")
-  )
-  (symbol (lib_id "SHT31V01A-rescue:R") (at 72.39 173.99 90) (unit 1)
-    (in_bom yes) (on_board yes)
-    (property "Reference" "R16" (id 0) (at 72.39 178.308 90))
-    (property "Value" "100R" (id 1) (at 72.39 173.99 90))
-    (property "Footprint" "Resistor_SMD:R_0603_1608Metric" (id 2) (at 72.39 175.768 90)
-      (effects (font (size 1.27 1.27)) hide)
-    )
-    (property "Datasheet" "" (id 3) (at 72.39 173.99 0))
-    (property "UST_ID" "5c70984512875079b91f8956" (id 4) (at 72.39 173.99 0)
-      (effects (font (size 1.27 1.27)) hide)
-    )
-    (pin "1")
-    (pin "2")
-  )
-  (symbol (lib_id "Device:R") (at 111.76 168.91 90) (unit 1)
-    (in_bom yes) (on_board yes)
-    (property "Reference" "R17" (id 0) (at 118.2116 167.767 90)
-      (effects (font (size 1.27 1.27)) (justify left))
-    )
-    (property "Value" "33R" (id 1) (at 113.538 169.037 90)
-      (effects (font (size 1.27 1.27)) (justify left))
-    )
-    (property "Footprint" "Resistor_SMD:R_0603_1608Metric" (id 2) (at 111.76 170.688 90)
-      (effects (font (size 1.27 1.27)) hide)
-    )
-    (property "Datasheet" "~" (id 3) (at 111.76 168.91 0)
-      (effects (font (size 1.27 1.27)) hide)
-    )
-    (property "UST_ID" "5c70984512875079b91f8952" (id 4) (at 111.76 168.91 0)
-      (effects (font (size 1.27 1.27)) hide)
-    )
-    (pin "1")
-    (pin "2")
-  )
-  (symbol (lib_id "Device:R") (at 111.76 171.45 90) (unit 1)
-    (in_bom yes) (on_board yes)
-    (property "Reference" "R18" (id 0) (at 118.2116 170.307 90)
-      (effects (font (size 1.27 1.27)) (justify left))
-    )
-    (property "Value" "33R" (id 1) (at 113.538 171.577 90)
-      (effects (font (size 1.27 1.27)) (justify left))
-    )
-    (property "Footprint" "Resistor_SMD:R_0603_1608Metric" (id 2) (at 111.76 173.228 90)
-      (effects (font (size 1.27 1.27)) hide)
-    )
-    (property "Datasheet" "~" (id 3) (at 111.76 171.45 0)
-      (effects (font (size 1.27 1.27)) hide)
-    )
-    (property "UST_ID" "5c70984512875079b91f8952" (id 4) (at 111.76 171.45 0)
-      (effects (font (size 1.27 1.27)) hide)
-    )

Commit message: Edit schema
Parts:
- added L?: L, symbol Device:L
Connections:
- net SD_VDD: now also L?.2; no longer U10.41 ((PCINT9/CLKO/T1)PB1), U10.42 ((PCINT10/AIN0/INT2)PB2), U10.43 ((PCINT11/AIN1/OC0)PB3)
- net POWER_ANALOG_3V3: now reaches U10.16 ((PCINT31/OC2A)PD7)
- net +5V renamed UAV_5V
- new net: L?.1, U10.41 ((PCINT9/CLKO/T1)PB1), U10.42 ((PCINT10/AIN0/INT2)PB2), U10.43 ((PCINT11/AIN1/OC0)PB3)
- no-connect marks 16 -> 15
Changed lines of the file:
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@@
   (no_connect (at 173.99 99.06))
   (no_connect (at 173.99 101.6))
-  (no_connect (at 173.99 124.46))
   (no_connect (at 261.62 133.35))
   (no_connect (at 261.62 137.16))
@@
     (stroke (width 0) (type default) (color 0 0 0 0))
   )
+  (wire (pts (xy 118.11 164.465) (xy 120.015 164.465))
+    (stroke (width 0) (type default) (color 0 0 0 0))
+  )
   (wire (pts (xy 119.38 26.67) (xy 119.38 25.4))
     (stroke (width 0) (type default) (color 0 0 0 0))
@@
     (stroke (width 0) (type default) (color 0 0 0 0))
   )
-  (wire (pts (xy 120.015 163.195) (xy 120.015 166.37))
-    (stroke (width 0) (type solid) (color 0 0 0 0))
+  (wire (pts (xy 120.015 164.465) (xy 120.015 166.37))
+    (stroke (width 0) (type default) (color 0 0 0 0))
   )
   (wire (pts (xy 120.65 179.07) (xy 120.65 181.61))
@@
     (stroke (width 0) (type default) (color 0 0 0 0))
   )
+  (wire (pts (xy 173.99 124.46) (xy 176.53 124.46))
+    (stroke (width 0) (type default) (color 0 0 0 0))
+  )
   (wire (pts (xy 176.53 63.5) (xy 176.53 66.04))
     (stroke (width 0) (type default) (color 0 0 0 0))
@@
     (stroke (width 0) (type default) (color 0 0 0 0))
   )
-  (wire (pts (xy 176.53 66.04) (xy 179.07 66.04))
+  (wire (pts (xy 176.53 66.04) (xy 182.88 66.04))
     (stroke (width 0) (type default) (color 0 0 0 0))
   )
@@
   )
   (wire (pts (xy 176.53 116.84) (xy 173.99 116.84))
+    (stroke (width 0) (type default) (color 0 0 0 0))
+  )
+  (wire (pts (xy 191.77 66.04) (xy 190.5 66.04))
     (stroke (width 0) (type default) (color 0 0 0 0))
   )
@@
     (effects (font (size 1.27 1.27)) (justify left bottom))
   )
-  (label "SD_VDD" (at 179.07 66.04 0)
+  (label "SD_VDD" (at 191.77 66.04 0)
     (effects (font (size 1.524 1.524)) (justify left bottom))
   )
@@
   (label "PC0" (at 252.73 63.5 0)
     (effects (font (size 1.524 1.524)) (justify left bottom))
+  )
+  (global_label "UAV_5V" (shape output) (at 118.11 164.465 180) (fields_autoplaced)
+    (effects (font (size 1.524 1.524)) (justify right))
+    (property "Intersheet References" "${INTERSHEET_REFS}" (id 0) (at 107.1931 164.3698 0)
+      (effects (font (size 1.524 1.524)) (justify right) hide)
+    )
   )
   (global_label "PA0" (shape input) (at 176.53 38.1 0) (fields_autoplaced)
@@
     )
   )
+  (global_label "POWER_ANALOG_3V3" (shape output) (at 176.53 124.46 0) (fields_autoplaced)
+    (effects (font (size 1.524 1.524)) (justify left))
+    (property "Intersheet References" "${INTERSHEET_REFS}" (id 0) (at 202.1789 124.3648 0)
+      (effects (font (size 1.524 1.524)) (justify left) hide)
+    )
+  )
   (symbol (lib_id "power:+3.3V") (at 17.78 88.9 0) (unit 1)
     (in_bom yes) (on_board yes)
@@
     )
     (property "Datasheet" "" (id 3) (at 119.38 25.4 0)
-      (effects (font (size 1.27 1.27)) hide)
-    )
-    (pin "1")
-  )
-  (symbol (lib_id "power:+5V") (at 120.015 163.195 0) (unit 1)
-    (in_bom yes) (on_board yes) (fields_autoplaced)
-    (property "Reference" "#PWR0126" (id 0) (at 120.015 167.005 0)
-      (effects (font (size 1.27 1.27)) hide)
-    )
-    (property "Value" "+5V" (id 1) (at 120.015 159.6476 0))
-    (property "Footprint" "" (id 2) (at 120.015 163.195 0)
-      (effects (font (size 1.27 1.27)) hide)
-    )
-    (property "Datasheet" "" (id 3) (at 120.015 163.195 0)
       (effects (font (size 1.27 1.27)) hide)
     )
@@
       (effects (font (size 1.27 1.27)) hide)
     )
+    (pin "1")
+    (pin "2")
+  )
+  (symbol (lib_id "Device:L") (at 186.69 66.04 90) (unit 1)
+    (in_bom yes) (on_board yes) (fields_autoplaced)
+    (property "Reference" "L?" (id 0) (at 186.69 61.5654 90))
+    (property "Value" "L" (id 1) (at 186.69 64.3405 90))
+    (property "Footprint" "" (id 2) (at 186.69 66.04 0)
+      (effects (font (size 1.27 1.27)) hide)
+    )
+    (property "Datasheet" "~" (id 3) (at 186.69 66.04 0)
+      (effects (font (size 1.27 1.27)) hide)
+    )

Commit message: Clean repository
Other:
- company: (none) -> UST
