File: hw/sch_pcb/SPACEDOS02B_PCB01A/cpu.kicad_sch (KiCad schematic)
At the start: 38 parts, among them J1 SM08B-GHS-TB, J10 HEADER_1x01, J11 HEADER_1x01, J12 HEADER_1x01, J13 HEADER_1x01, J14 SM06B-GHS-TB, J19 HEADER_2x01_PARALLEL, J22 HEADER_2x03, J4 HEADER_1x01, J5 HEADER_1x01, J6 HEADER_1x01, J7 HEADER_1x01, J8 HEADER_1x01, J9 HEADER_1x01, U10 ATMEGA1284P-AU, U11 PCF85263A, U6 AT24CS64-SSHM, Y1 1,8432MHz, Y2 ABS07-120-32.768KHZ-T

Commit message: clean repository
Parts:
- gave numbers to parts that had none: 1
Changed lines of the file:
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@@
   (symbol (lib_id "Device:L") (at 186.69 66.04 90) (unit 1)
     (in_bom yes) (on_board yes) (fields_autoplaced)
-    (property "Reference" "L?" (id 0) (at 186.69 61.5654 90))
+    (property "Reference" "L2" (id 0) (at 186.69 61.5654 90))
     (property "Value" "L" (id 1) (at 186.69 64.3405 90))
     (property "Footprint" "" (id 2) (at 186.69 66.04 0)
