File: hw/sch_pcb/SPACEDOS02B_PCB01A/SPACEDOS02B_PCB01A.kicad_pcb (KiCad board)
At the start: 2 copper layers, 38 x 200 mm, 120 parts, among them J1 MCC-SD, J10 HEADER_1x01, J11 HEADER_1x01, J12 HEADER_1x01, J13 HEADER_1x01, J14 HEADER_1x01, J15 HEADER_1x01, J16 HEADER_1x01, J17 HEADER_1x01, J18 HEADER_1x01, J19 HEADER_2x01_PARALLEL, J2 HEADER_2x01_PARALLEL, J20 HEADER_1x01, J21 HEADER_1x01, J22 HEADER_2x03, J23 HEADER_1x01, J24 HEADER_1x01, J25 HEADER_1x01, J26 HEADER_1x01, J27 HEADER_1x01, J28 SD_Card-FPS009-4200-0, J3 HEADER_2x01_PARALLEL, J4 HEADER_1x01, J5 HEADER_1x01, J6 HEADER_1x01, J7 HEADER_1x01, J8 HEADER_1x01, J9 HEADER_1x01, M6 BMI-S-210-F, M8 BMI-S-210-F, U1 OPA2314, U10 ATMEGA1284P-AU, U11 PCF85263A, U2 OPA2314, U3 ISL21080DIH312Z-TK 1V25, U4 TS7211, U5 TS5A4594, U6 AT24CS64-SSHM, U8 TPS613222ADBV, Y2 ABS07-120-32.768KHZ-T

Commit message: Oprava otvíratelnosti schéma.
Parts:
- added U7: IR4302, Package_DFN_QFN:Infineon_PQFN-44-31-5EP_7x7mm_P0.5mm, F.Cu at (75.3, -108.5)

Commit message: #4 add crystal
Parts:
- removed U7: IR4302, Package_DFN_QFN:Infineon_PQFN-44-31-5EP_7x7mm_P0.5mm
- added C38: 15pF, Mlab_R:SMD-0805, B.Cu at (68.4, -63.4)
- added C41: 15pF, Mlab_R:SMD-0805, B.Cu at (72.5, -63.4)
- added Y1: 1,8432MHz, Crystal:Crystal_HC49-U_Horizontal, F.Cu at (19.5, -56.7)
- moved C30 0.90 mm to (12.3, -53.4)
Connections:
- U10 pad 7: unconnected-(U10-Pad7) -> Net-(U10-Pad7)
- U10 pad 8: unconnected-(U10-Pad8) -> Net-(U10-Pad8)
Routing:
- net +3V3: track 198.0 -> 210.8 mm
- net /cpu/RST#_P: track 12.8 -> 0.00 mm
- net PA0: vias 2 -> 3
- net GND: vias 233 -> 232

Commit message: Edit PCB
Parts:
- removed C22, C33: 10uF, Mlab_R:SMD-0805
- removed C25, C37: 100nF, Mlab_R:SMD-0805
- removed J1: MCC-SD, Mlab_CON:MCC-SD
- removed J14, J15, J16, J17, J18, J20, J21, J23, J24, J25, J26, J27: HEADER_1x01, Mlab_Pin_Headers:Straight_1x01
- removed J28: SD_Card-FPS009-4200-0, Mlab_CON:FPS009-4200-0
- removed R14, R16, R17, R18, R24, R25, R26, R27: 100, Mlab_R:SMD-0805
Routing:
- net GND: track 99.8 -> 72.5 mm
- net Net-(J14-Pad1): track 22.2 -> 0.00 mm
- net /cpu/SD_VDD2: track 20.9 -> 0.00 mm, vias 1 -> 0
- net Net-(J21-Pad1): track 19.5 -> 0.00 mm
- net Net-(J15-Pad1): track 16.9 -> 0.00 mm
- net /cpu/SD_VDD3: track 16.2 -> 0.00 mm, vias 1 -> 0
- net Net-(J23-Pad1): track 14.4 -> 0.00 mm
- net Net-(J26-Pad1): track 10.4 -> 0.00 mm
- net Net-(J18-Pad1): track 8.93 -> 0.00 mm
- net Net-(J25-Pad1): track 7.71 -> 0.00 mm
- net Net-(J17-Pad1): track 7.36 -> 0.00 mm
- net Net-(J28-Pad1): track 2.49 -> 0.00 mm
- net Net-(J28-Pad2): track 2.47 -> 0.00 mm
- net Net-(J28-Pad7): track 2.45 -> 0.00 mm
- net Net-(J28-Pad5): track 2.42 -> 0.00 mm
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Other:
- board size 38 x 200 mm -> 38 x 110 mm

Commit message: Edit schema
Parts:
- added J1: SM08B-GHS-TB, Connector_JST:JST_GH_SM08B-GHS-TB_1x08-1MP_P1.25mm_Horizontal, F.Cu at (75.7, -88.6)
- added J14: SM06B-GHS-TB, Connector_JST:JST_GH_SM06B-GHS-TB_1x06-1MP_P1.25mm_Horizontal, F.Cu at (56.6, -61.8)
- added R14: 100R, Resistor_SMD:R_0603_1608Metric, F.Cu at (85.4, -91.1)
- added R16: 100R, Resistor_SMD:R_0603_1608Metric, F.Cu at (79.5, -85.2)
- added R17: 33R, Resistor_SMD:R_0603_1608Metric, F.Cu at (47.9, -58.4)
- added R18: 33R, Resistor_SMD:R_0603_1608Metric, F.Cu at (48.0, -60.6)

Commit message: Edit
Parts:
- moved J1 72.2 mm to (4.98, -73.9), turned to -90 degrees
- moved J14 50.0 mm to (6.65, -59.8), turned to -90 degrees
Connections:
- U10 pad 11: unconnected-(U10-Pad11) -> /cpu/RX1
- U10 pad 12: unconnected-(U10-Pad12) -> /cpu/TX1
- U10 pad 13: unconnected-(U10-Pad13) -> /cpu/TIMEPULSE
- U10 pad 14: unconnected-(U10-Pad14) -> /cpu/EXTINT
- U10 pad 15: unconnected-(U10-Pad15) -> /cpu/GEO_STAT
Routing:
- net +3V3: track 210.8 -> 211.7 mm
- net GND: vias 232 -> 231
- net /cpu/RX1: vias 0 -> 1

Commit message: Clean repository
Parts:
- moved BT1 197.8 mm to (114.3, 112.6)
- moved C1 197.8 mm to (125.0, 145.8)
- moved C10 197.8 mm to (117.4, 163.0)
- moved C11 197.8 mm to (117.7, 155.6)
- moved C12 197.8 mm to (116.4, 135.5)
- moved C13 197.8 mm to (108.3, 137.8)
- moved C14 197.8 mm to (124.4, 130.6)
- moved C15 197.8 mm to (113.9, 153.1)
- moved C16 197.8 mm to (113.8, 151.0)
- moved C17 197.8 mm to (111.5, 143.5)
- moved C18 197.8 mm to (117.5, 146.2)
- moved C19 197.8 mm to (112.6, 135.5)
- moved C2 197.8 mm to (106.7, 153.0)
- moved C20 197.8 mm to (121.7, 163.2)
- moved C21 197.8 mm to (106.7, 148.9)
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
Commit message: clean repository
Parts:
- removed R14, R16: 100R, Resistor_SMD:R_0603_1608Metric
- removed R17, R18: 33R, Resistor_SMD:R_0603_1608Metric
- added U7: MIC5504-3.3YM5, Package_TO_SOT_SMD:SOT-23-5, F.Cu at (126.1, 50.6)
Connections:
- C1 pad 1: +3V3 -> POWER_ANALOG_3V3
- C32 pad 1: +3V3 -> POWER_ANALOG_3V3
- C4 pad 1: +3V3 -> POWER_ANALOG_3V3
- J1 pad 4: Net-(J1-Pad4) -> /cpu/PC1
- J1 pad 5: Net-(J1-Pad5) -> /cpu/PC0
- J14 pad 1: +5V -> UAV_5V
- J14 pad 2: Net-(J14-Pad2) -> /cpu/RX0
- J14 pad 3: Net-(J14-Pad3) -> /cpu/TX0
- L3 pad 1: +3V3 -> POWER_ANALOG_3V3
- R2 pad 2: +3V3 -> POWER_ANALOG_3V3
- R3 pad 2: +3V3 -> POWER_ANALOG_3V3
- R4 pad 2: +3V3 -> POWER_ANALOG_3V3
- R5 pad 2: +3V3 -> POWER_ANALOG_3V3
- U10 pad 16: unconnected-(U10-Pad16) -> POWER_ANALOG_3V3
- U10 pad 41: /cpu/SD_VDD -> Net-(U10-Pad41)
- U10 pad 42: /cpu/SD_VDD -> Net-(U10-Pad41)
- U10 pad 43: /cpu/SD_VDD -> Net-(U10-Pad41)
- U3 pad 1: +3V3 -> POWER_ANALOG_3V3
Routing:
- net POWER_ANALOG_3V3: track 0.00 -> 42.8 mm, vias 0 -> 3
- net +3V3: track 211.7 -> 168.9 mm, vias 6 -> 3
- net Net-(U10-Pad41): track 0.00 -> 10.0 mm, vias 0 -> 1
- net /cpu/SD_VDD: track 55.8 -> 45.7 mm, vias 1 -> 0
- net PA0: vias 3 -> 2
- net /cpu/RX1: vias 1 -> 2
