File: hw/sch_pcb/SPACEDOS02B_PCB01A/power.kicad_sch (KiCad schematic)
At the start: 15 parts, among them J2 HEADER_2x01_PARALLEL, J3 HEADER_2x01_PARALLEL, U8 TPS613222ADBV

Commit message: Edit schema
Parts:
- added C?: 10uF, Mlab_R:SMD-0805, symbol Device:C
- added C?: 1uF, Mlab_R:SMD-0603, symbol Device:C
- added C?: 100nF, Mlab_R:SMD-0603, symbol Device:C
- added U?: MIC5504-3.3YM5, Package_TO_SOT_SMD:SOT-23-5, symbol Regulator_Linear:MIC5504-3.3YM5
Connections:
- net +3V3: no longer C32.1, L3.1
- net 3: now also C?.1, U?.5 (VOUT)
- net GND: now also C?.2, C?.2, C?.2, U?.2 (GND)
- new net POWER_ANALOG_3V3: C32.1, L3.1
- new net UAV_5V: C?.1, C?.1, U?.1 (VIN), U?.3 (EN)
Other:
- moved on the sheet: BT1, C29, C32, C36, C42, C50, C52, C54, C55, D3, F2, J2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

Commit message: Clean repository
Other:
- company: (none) -> UST

Commit message: clean repository
Parts:
- gave numbers to parts that had none: 4
Changed lines of the file:
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@@
   (symbol (lib_id "Device:C") (at 36.83 114.935 0) (unit 1)
     (in_bom yes) (on_board yes)
-    (property "Reference" "C?" (id 0) (at 36.83 112.395 0)
+    (property "Reference" "C22" (id 0) (at 36.83 112.395 0)
       (effects (font (size 1.27 1.27)) (justify left))
     )
@@
   (symbol (lib_id "power:GND") (at 66.675 122.555 0) (unit 1)
     (in_bom yes) (on_board yes)
-    (property "Reference" "#PWR?" (id 0) (at 66.675 128.905 0)
+    (property "Reference" "#PWR0106" (id 0) (at 66.675 128.905 0)
       (effects (font (size 1.27 1.27)) hide)
     )
@@
   (symbol (lib_id "Device:C") (at 80.645 114.935 0) (unit 1)
     (in_bom yes) (on_board yes)
-    (property "Reference" "C?" (id 0) (at 83.566 113.7666 0)
+    (property "Reference" "C33" (id 0) (at 83.566 113.7666 0)
       (effects (font (size 1.27 1.27)) (justify left))
     )
@@
   (symbol (lib_id "Device:C") (at 44.45 114.935 0) (unit 1)
     (in_bom yes) (on_board yes)
-    (property "Reference" "C?" (id 0) (at 44.45 112.395 0)
+    (property "Reference" "C25" (id 0) (at 44.45 112.395 0)
       (effects (font (size 1.27 1.27)) (justify left))
     )
@@
   (symbol (lib_id "power:GND") (at 80.645 122.555 0) (unit 1)
     (in_bom yes) (on_board yes)
-    (property "Reference" "#PWR?" (id 0) (at 80.645 128.905 0)
+    (property "Reference" "#PWR0107" (id 0) (at 80.645 128.905 0)
       (effects (font (size 1.27 1.27)) hide)
     )
@@
   (symbol (lib_id "Regulator_Linear:MIC5504-3.3YM5") (at 66.675 111.125 0) (unit 1)
     (in_bom yes) (on_board yes)
-    (property "Reference" "U?" (id 0) (at 66.675 101.8032 0))
+    (property "Reference" "U7" (id 0) (at 66.675 101.8032 0))
     (property "Value" "MIC5504-3.3YM5" (id 1) (at 66.675 104.1146 0))
     (property "Footprint" "Package_TO_SOT_SMD:SOT-23-5" (id 2) (at 66.675 121.285 0)
@@
   (symbol (lib_id "power:GND") (at 36.83 122.555 0) (unit 1)
     (in_bom yes) (on_board yes)
-    (property "Reference" "#PWR?" (id 0) (at 36.83 128.905 0)
+    (property "Reference" "#PWR0126" (id 0) (at 36.83 128.905 0)
       (effects (font (size 1.524 1.524)) hide)
     )
