File: hw/sch_pcb/SPACEDOS02B_PCB02A/SPACEDOS02B_PCB02A.kicad_pcb (KiCad board)
At the start: 2 copper layers, 38 x 50 mm, 14 parts, among them J21 HEADER_1x01, J23 HEADER_1x01, J24 HEADER_1x01, J25 HEADER_1x01, J26 HEADER_1x01, J27 HEADER_1x01, J28 SD_Card-FPS009-4200-0

Commit message: Clean repository
Parts:
- moved G*** 288.7 mm to (137.2, 88.0)
- moved J21 288.7 mm to (146.5, 66.6)
- moved J24 288.7 mm to (149.0, 66.6)
- moved J25 288.7 mm to (138.9, 66.6)
- moved J26 288.7 mm to (141.4, 66.6)
- moved J27 288.7 mm to (151.6, 66.6)
- moved J28 288.7 mm to (139.1, 112.8)
- moved R24 288.7 mm to (133.5, 73.2)
- moved R25 288.7 mm to (136.1, 73.2)
- moved R26 288.7 mm to (143.7, 73.2)
- moved R27 288.7 mm to (148.8, 73.2)
- moved C33 288.7 mm to (140.1, 71.2)
- moved C37 288.7 mm to (140.1, 73.7)
- moved J23 288.7 mm to (144.0, 66.6)
