File: hw/sch_pcb/SPACEDOS02B_PCB02A/SPACEDOS02B_PCB02A.kicad_sch (KiCad schematic)
At the start: 0 parts

Commit message: Clean repository
Other:
- company: Mlab www.mlab.cz -> UST
- title: NAME -> SPACEDOS02B - PCB02A
Changed lines of the file:
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@@
-(kicad_sch (version 20210621) (generator eeschema)
+(kicad_sch (version 20211123) (generator eeschema)
   (paper "A4")
   (title_block
-    (title "NAME")
+    (title "SPACEDOS02B - PCB02A")
     (date "%F")
-    (rev "REV")
-    (company "Mlab www.mlab.cz")
-    (comment 1 "VERSION")
-    (comment 2 "Short description \\nTwo lines are maximum")
-    (comment 3 "nickname <email@example.com>")
-    (comment 4 "BSD")
+    (company "UST")
   )
   (sheet (at 142.24 83.82) (size 21.59 8.89) (fields_autoplaced)
     (stroke (width 0) (type solid) (color 0 0 0 0))
     (fill (color 0 0 0 0.0000))
-    (property "Název listu" "cpu" (id 0) (at 142.24 82.9814 0)
+    (property "Sheet name" "cpu" (id 0) (at 142.24 82.9814 0)
       (effects (font (size 1.524 1.524)) (justify left bottom))
     )
-    (property "Soubor listu" "cpu.kicad_sch" (id 1) (at 142.24 93.3962 0)
+    (property "Sheet file" "cpu.kicad_sch" (id 1) (at 142.24 93.3962 0)
       (effects (font (size 1.524 1.524)) (justify left top))
     )
