File: hw/sch_pcb/SPACEDOS02B_PCB02A/cpu.kicad_sch (KiCad schematic)
At the start: 13 parts, among them J21 HEADER_1x01, J23 HEADER_1x01, J24 HEADER_1x01, J25 HEADER_1x01, J26 HEADER_1x01, J27 HEADER_1x01, J28 SD_Card-FPS009-4200-0

Commit message: Clean repository
Other:
- company: (none) -> UST
- title: (none) -> SPACEDOS02B - PCB02A
